File: motor-controller-hw/motor-controller-hw.sch (KiCad schematic (older format))
At the start: 0 parts

Commit message: Added system library parts to project library Added a few more comments to IO.sch Added TMC4671 SPI bus as an output for microcontroller.sch Added some connections in the overview page Updated schematic dates
Connections:
- wire segments 28 -> 47
Changed lines of the file:
@@
 Sheet 1 5
 Title "Motor Controller Control Board"
-Date ""
-Rev ""
+Date "2018-11-17"
+Rev "1.0"
 Comp "Cedarville University"
 Comment1 "Supermileage Motor Controller"
@@
 L MotorControllerParts:GNDD #PWR0111
 U 1 1 5BB25C8D
-P 5150 5900
-F 0 "#PWR0111" H 5150 5650 50  0001 C CNN
-F 1 "GNDD" H 5150 5750 50  0000 C CNN
-F 2 "" H 5150 5900 50  0001 C CNN
-F 3 "" H 5150 5900 50  0001 C CNN
-	1    5150 5900
+P 3800 5400
+F 0 "#PWR0111" H 3800 5150 50  0001 C CNN
+F 1 "GNDD" H 3800 5250 50  0000 C CNN
+F 2 "" H 3800 5400 50  0001 C CNN
+F 3 "" H 3800 5400 50  0001 C CNN
+	1    3800 5400
 	1    0    0    -1
 $EndComp
@@
 $EndComp
 Wire Wire Line
-	5150 5900 5150 5800
-Wire Wire Line
-	5150 5800 5300 5800
+	3800 5400 3800 5150
+Wire Wire Line
+	3800 5150 3950 5150
 Wire Wire Line
 	3150 1850 3150 1750
@@
 vBat
 $Sheet
-S 4000 2800 1850 2350
+S 3950 2950 1850 2300
 U 5BE2BA0F
 F0 "STM32" 50
 F1 "microcontroller.sch" 50
-F2 "3.3v" I L 4000 2900 50
+F2 "3.3v" I L 3950 3050 50
+F3 "USB_D+" B L 3950 3200 50
+F4 "USB_D-" B L 3950 3300 50
+F5 "CAN_Rx" B L 3950 3450 50
+F6 "CAN_Tx" B L 3950 3550 50
+F7 "Throttle" I L 3950 3700 50
+F8 "MotorTemp" I L 3950 3800 50
+F9 "TransistorTemp" I L 3950 3900 50
+F10 "A_In1" I L 3950 4050 50
+F11 "A_In2" I L 3950 4150 50
+F12 "D_In1" I L 3950 4250 50
+F13 "D_In2" I L 3950 4350 50
+F14 "D_In3" I L 3950 4450 50
+F15 "D_In4" I L 3950 4550 50
+F16 "A_Out1" O L 3950 4700 50
+F17 "A_Out2" O L 3950 4800 50
+F18 "D_Out1" O L 3950 4900 50
+F19 "D_Out2" O L 3950 5000 50
+F20 "DGND" I L 3950 5150 50
+F21 "TMC4671_SS" O R 5800 3550 50
+F22 "TMC4671_SCK" O R 5800 3650 50
+F23 "TMC4671_MISO" I R 5800 3750 50
+F24 "TMC4671_MOSI" I R 5800 3850 50
 $EndSheet
 $Sheet
@@
 F51 "TMC4671_Tx_i" I L 1600 2950 50
 $EndSheet
+Wire Wire Line
+	3000 4050 3950 4050
+Wire Wire Line
+	3000 4150 3950 4150
+Wire Wire Line
+	3000 4250 3950 4250
+Wire Wire Line
+	3000 4350 3950 4350
+Wire Wire Line
+	3950 4450 3000 4450
+Wire Wire Line
+	3000 4550 3950 4550
+Wire Wire Line
+	3000 4700 3950 4700
+Wire Wire Line
+	3000 4800 3950 4800
+Wire Wire Line
+	3000 4900 3950 4900
+Wire Wire Line
+	3000 5000 3950 5000
+Wire Wire Line
+	3000 3900 3950 3900
+Wire Wire Line
+	3000 3800 3950 3800
+Wire Wire Line
+	3000 3700 3950 3700
+Wire Wire Line
+	3000 3550 3950 3550
+Wire Wire Line
+	3000 3450 3950 3450
+Wire Wire Line
+	3000 3300 3950 3300
+Wire Wire Line
+	3000 3200 3950 3200
+$Comp
+L MotorControllerParts:+3.3V #PWR?
+U 1 1 5BF2523A
+P 3800 2800
+F 0 "#PWR?" H 3800 2650 50  0001 C CNN
+F 1 "+3.3V" H 3815 2973 50  0000 C CNN
+F 2 "" H 3800 2800 50  0001 C CNN
+F 3 "" H 3800 2800 50  0001 C CNN
+	1    3800 2800
+	1    0    0    -1
+$EndComp
+Wire Wire Line
+	3800 3050 3950 3050
+Wire Wire Line
+	3800 2800 3800 3050
 $EndSCHEMATC

Commit message: motor-controller-hw.sch: Added power supply to the top level schematic Added connectors for all the IO pins
Parts:
- added C?: 100n, symbol MotorControllerParts:C
- added C? (x2): 4u7, symbol MotorControllerParts:C
- added C?: 10u, symbol MotorControllerParts:C
- added C?: 33u, symbol MotorControllerParts:C
- added D?: 18V Zener, symbol Device:D_Zener_ALT
- added F?: 50mA PTC, symbol Device:Polyfuse_Small
- added J?: Hall Sensors, symbol Connector_Generic:Conn_01x06
- added J?: USB_B_Micro, symbol Connector:USB_B_Micro
- added J?: CAN1, symbol Connector_Generic:Conn_01x04
- added J?: Motor Temp, symbol Connector_Generic:Conn_01x02
- added J?: Transistor Temp, symbol Connector_Generic:Conn_01x02
- added J?: Throttle, symbol Connector_Generic:Conn_01x04
- added J?: Extra IO, symbol Connector_Generic:Conn_02x07_Top_Bottom
- added Q?: Q_PMOS_GDS, symbol Device:Q_PMOS_GDS
- added R? (x2): 10K, symbol MotorControllerParts:R
- added U?: D36V6F5, supermileage_footprints:D36V6Fx, symbol MotorControllerParts:D36V6Fx
- added U?: AP7361C-33, TO_SOT_Packages_SMD:SOT-223, symbol MotorControllerParts:AP7361C
Connections:
- net labels added: A_Out1, A_Out2, A_in1, A_in2, CAN_H, CAN_L, D_Out1, D_Out2, D_in1, D_in2, D_in3, D_in4, Hall1, Hall2, Hall3, MotorTemp, Throttle, TransistorTemp, USB_D+, USB_D-, Vin
- wire segments 47 -> 148
- no-connect marks 0 -> 2
Other:
- note added: "3.3V linear voltage regulator for the low voltage electronics. The selected\nregulator can supply 1A of output current, which is more than what the 5V \nswitching regulator can supply. The 4.7uF output capacitor should have a \nfairly low ESR."
- note added: "5V switching regulator, up to 50V input, maximum 600mA output current. \nP-Channel MOSFET for an ideal diode with a 18v zener diode to protect the \nMOSFET gate. The 10K resistor limits the zener diode current to 3mA at \n48V input."

Commit message: Moving away from TMC4671
Parts:
- added J?: Trinamic-Conntector, symbol MotorControllerParts:Trinamic-Conntector
Connections:
- net labels added: ADC_I_A, ADC_I_B, Batt_Current, HallA, HallA_FX_in, HallA_in, HallB, HallB_FX_in, HallB_in, HallC, HallC_FX_in, HallC_in, PWM_AH, PWM_AL, PWM_BH, PWM_BL, PWM_CH, PWM_CL, PWM_Idle_H, PWM_Idle_L
- net labels removed: D_GND, GNDPWR, Hall1, Hall2, Hall3, PWM_Phase_AH, PWM_Phase_AL, PWM_Phase_BH, PWM_Phase_BL, PWM_Phase_CH, PWM_Phase_CL, P_GND, Phase_A_Current, Phase_A_HALFX, Phase_B_Current, Phase_B_HALFX, Phase_C_Current, Phase_C_HALFX, vBat
- wire segments 148 -> 180

Commit message: Voltage regualtor changes, name changes, and HANDS!!!
Parts:
- added D?: D_USB, symbol Device:D_Schottky_ALT
- added F? (x2): 50mA PTC, symbol Device:Polyfuse_Small
- added J?: CAN_DBG, symbol Connector_Generic:Conn_01x02
- added J?: SPI_DBG, symbol Connector_Generic:Conn_01x04
- added J?: ABN_In, symbol Connector_Generic:Conn_01x05
- J?: value Trinamic-Conntector -> Trinamic-Bridge
Connections:
- net labels added: ENC_A, ENC_A_in, ENC_B, ENC_B_in, ENC_N, ENC_N_in, En_Out, PWM_DH, PWM_DL, V_USB
- net labels removed: HallA_FX_in, HallB_FX_in, HallC_FX_in
- wire segments 180 -> 227
Other:
- note added: "5V switching regulator, up to 50V input, maximum 600mA output current. \nThe regulator is short circuit protected.\nA P-Channel MOSFET is used as an ideal diode with a 18v zener diode to\nprotect the MOSFET gate. The 10K resistor limits the zener diode current\nto 3mA at 48V input. A Shocktty diode is used to protect the USB 5V line\nfrom reverse current."
- note removed: "5V switching regulator, up to 50V input, maximum 600mA output current. \nP-Channel MOSFET for an ideal diode with a 18v zener diode to protect the \nMOSFET gate. The 10K resistor limits the zener diode current to 3mA at \n48V input."

Commit message: Working schematics
Parts:
- added TP? (x2): 5v_TP, symbol MotorControllerParts:TestPoint_2Pole
- added TP?: 3v3_TP, symbol MotorControllerParts:TestPoint_2Pole
- added TP? (x2): GND_TP, symbol MotorControllerParts:TestPoint
Connections:
- net labels added: Brake_Chopper
- wire segments 227 -> 237
- no-connect marks 2 -> 3
Other:
- note added: "PWM_Ax, PWM_Bx, and PWM_Cx correspond to the A, B, and C phases of\na three phase motor. The PWM_Dx lines are for a "extra" fourth phase.\nNote that the A, B, and C lines may be labeled U, V, and W elsewhere which\nare their european designation."
- note added: "Power supply test points"
- note added: "Remember the golden rule of debugging:\n**Thou Shalt Measure Voltages**\nThese points have been provided for your\nmeasurement convienence."

Commit message: Compacted schematic layout
Parts:
- J101: renamed from J?; value CAN1 -> CAN
- J109: renamed from J?; value ABN_In -> ABN Encoder
- gave numbers to parts that had none: 29
Connections:
- net labels added: Brake
- net labels removed: Brake_Chopper
- wire segments 237 -> 236
Other:
- note added: "Analog IO"
- note added: "Digital Comm"
- note added: "Encoders"
- note added: "PWM_Ax, PWM_Bx, and PWM_Cx correspond to the A, B, and C phases of\na three phase motor. The PWM_Dx lines are for a "extra" fourth phase.\nNote that the A, B, and C lines may be labeled U, V, and W elsewhere \nwhich are their european designation."
- note removed: "PWM_Ax, PWM_Bx, and PWM_Cx correspond to the A, B, and C phases of\na three phase motor. The PWM_Dx lines are for a "extra" fourth phase.\nNote that the A, B, and C lines may be labeled U, V, and W elsewhere which\nare their european designation."
- note removed: "Remember the golden rule of debugging:\n**Thou Shalt Measure Voltages**\nThese points have been provided for your\nmeasurement convienence."

Commit message: Moved all parts into the MotorControllerParts.lib file
Parts:
- D102: symbol Device:D_Schottky_ALT -> MotorControllerParts:D_Schottky_ALT
- F101, F102, F103: symbol Device:Polyfuse_Small -> MotorControllerParts:Polyfuse_Small
- J101, J102, J110: symbol Connector_Generic:Conn_01x04 -> MotorControllerParts:Conn_01x04
- J103, J104, J108: symbol Connector_Generic:Conn_01x02 -> MotorControllerParts:Conn_01x02
- J105: symbol Connector:USB_B_Micro -> MotorControllerParts:USB_B_Micro
- J106: symbol Connector_Generic:Conn_02x07_Top_Bottom -> MotorControllerParts:Conn_02x07_Top_Bottom
- J107: symbol Connector_Generic:Conn_01x06 -> MotorControllerParts:Conn_01x06
- J109: symbol Connector_Generic:Conn_01x05 -> MotorControllerParts:Conn_01x05
Connections:
- net labels added: SPI_MISO, SPI_MOSI, SPI_SCK, SPI_SS
- wire segments 236 -> 245
- no-connect marks 3 -> 14
Changed lines of the file:
@@
 F25 "TMC4671_EN" O R 7650 4150 50
 F26 "TMC4671_Status" I R 7650 4250 50
+F27 "~SPI_SS" O R 7650 5250 50
+F28 "SPI_SCK" O R 7650 5150 50
+F29 "SPI_MISO" I R 7650 5050 50
+F30 "SPI_MOSI" O R 7650 4950 50
 $EndSheet
 Wire Wire Line
@@
 U 1 1 5BFA3D9B
 P 5650 1550
-F 0 "C102" H 5765 1596 50  0000 L CNN
-F 1 "100n" H 5765 1505 50  0000 L CNN
+F 0 "C102" H 5700 1650 50  0000 L CNN
+F 1 "100n" H 5700 1450 50  0000 L CNN
 F 2 "" H 5688 1400 50  0001 C CNN
 F 3 "" H 5650 1550 50  0001 C CNN
@@
 U 1 1 5BFA3DA9
 P 7600 1550
-F 0 "C105" H 7715 1596 50  0000 L CNN
+F 0 "C105" H 7650 1650 50  0000 L CNN
 F 1 "10u" H 7650 1450 50  0000 L CNN
 F 2 "" H 7638 1400 50  0001 C CNN
@@
 U 1 1 5BFA3DB0
 P 5250 1550
-F 0 "C101" H 5365 1596 50  0000 L CNN
-F 1 "4u7" H 5365 1505 50  0000 L CNN
+F 0 "C101" H 5300 1650 50  0000 L CNN
+F 1 "4u7" H 5300 1450 50  0000 L CNN
 F 2 "" H 5288 1400 50  0001 C CNN
 F 3 "" H 5250 1550 50  0001 C CNN
@@
 	5000 550  8000 550
 $Comp
-L Connector:USB_B_Micro J105
+L MotorControllerParts:USB_B_Micro J105
 U 1 1 5BFDD119
 P 900 1200
@@
 	850  1650 900  1650
 $Comp
-L Connector_Generic:Conn_01x04 J101
+L MotorControllerParts:Conn_01x04 J101
 U 1 1 5BFE5442
 P 800 2350
@@
 	1100 2450 1000 2450
 $Comp
-L Connector_Generic:Conn_01x02 J103
+L MotorControllerParts:Conn_01x02 J103
 U 1 1 5BFEEFEC
 P 800 4300
@@
 $EndComp
 $Comp
-L Connector_Generic:Conn_01x02 J104
+L MotorControllerParts:Conn_01x02 J104
 U 1 1 5BFF0D92
 P 800 5150
@@
 TransistorTemp
 $Comp
-L Connector_Generic:Conn_01x04 J102
+L MotorControllerParts:Conn_01x04 J102
 U 1 1 5C001BC1
 P 800 3550
@@
 $EndComp
 $Comp
-L Connector_Generic:Conn_02x07_Top_Bottom J106
+L MotorControllerParts:Conn_02x07_Top_Bottom J106
 U 1 1 5C00DFF5
 P 1400 6200
@@
 NoConn ~ 1000 2150
 $Comp
-L Device:Polyfuse_Small F101
+L MotorControllerParts:Polyfuse_Small F101
 U 1 1 5C1CAD40
 P 1350 3350
@@
 Connection ~ 1150 3350
 $Comp
-L Connector_Generic:Conn_01x06 J107
+L MotorControllerParts:Conn_01x06 J107
 U 1 1 5BF7BB3E
 P 2000 4950
@@
 	3100 1450 3800 1450
 $Comp
-L Device:D_Schottky_ALT D102
+L MotorControllerParts:D_Schottky_ALT D102
 U 1 1 5DE9991E
 P 2950 1450
@@
 U 1 1 5BFA3DF0
 P 2450 2350
-F 0 "R102" H 2250 2400 50  0000 L CNN
+F 0 "R102" H 2150 2400 50  0000 L CNN
 F 1 "10K" H 2200 2300 50  0000 L CNN
 F 2 "" V 2380 2350 50  0001 C CNN
@@
 	5400 6600 5100 6600
 $Comp
-L Device:Polyfuse_Small F103
+L MotorControllerParts:Polyfuse_Small F103
 U 1 1 5E1B011D
 P 1850 6000
@@
 $EndComp
 $Comp
-L Device:Polyfuse_Small F102
+L MotorControllerParts:Polyfuse_Small F102
 U 1 1 5E1C927F
 P 1850 5900
@@
 	8050 4000 8050 4750
 $Comp
-L Connector_Generic:Conn_01x02 J108
+L MotorControllerParts:Conn_01x02 J108
 U 1 1 5E6A4ACF
 P 5200 3800
@@
 $EndComp
 $Comp
-L Connector_Generic:Conn_01x04 J110
+L MotorControllerParts:Conn_01x04 J110
 U 1 1 5E6B408E
 P 7850 3800
@@
 ENC_A_in
 $Comp
-L Connector_Generic:Conn_01x05 J109
+L MotorControllerParts:Conn_01x05 J109
 U 1 1 5E777130
 P 2100 3550
@@
 Wire Notes Line
 	550  6750 550  5600
+Wire Wire Line
+	1700 5900 1750 5900
+Wire Wire Line
+	8050 5050 7650 5050
+Wire Wire Line
+	8050 4950 7650 4950
+Wire Wire Line
+	8050 5150 7650 5150
+Wire Wire Line
+	8050 5250 7650 5250
+Text Label 8050 4950 2    50   ~ 0
+SPI_MISO
+Text Label 8050 5050 2    50   ~ 0
+SPI_MOSI
+Text Label 8050 5150 2    50   ~ 0
+SPI_SCK
+Text Label 8050 5250 2    50   ~ 0
+SPI_SS
+Text Label 10450 1850 2    50   ~ 0
+SPI_MISO
+Text Label 10450 1650 2    50   ~ 0
+SPI_MOSI
+Text Label 10450 2050 2    50   ~ 0
+SPI_SS
+Text Label 8150 1850 0    50   ~ 0
+SPI_SCK
+Wire Wire Line
+	10450 2050 9900 2050
+Wire Wire Line
+	8150 1850 8650 1850
+Wire Wire Line
+	10450 1650 9900 1650
+Wire Wire Line
+	10450 1850 9900 1850
+NoConn ~ 9900 3050
+NoConn ~ 9900 2950
+NoConn ~ 9900 2850
+NoConn ~ 9900 2750
+NoConn ~ 9900 2650
+NoConn ~ 9900 1350
+NoConn ~ 8650 2950
+NoConn ~ 8650 2850
+NoConn ~ 8650 2750
+NoConn ~ 8650 2650
+NoConn ~ 8650 2550
 $EndSCHEMATC

Commit message: Added footprints, changed pdf
Parts:
- C101, C102, C104, C105: footprint (none) -> Capacitor_SMD:C_0805_2012Metric_Pad1.15x1.40mm_HandSolder
- J101, J102: footprint (none) -> supermileage_footprints:Molex-duraClick-4conn
- J108, TP101, TP102, TP103: footprint (none) -> Connector_PinHeader_2.54mm:PinHeader_1x02_P2.54mm_Vertical
- J109: footprint (none) -> Connector_PinHeader_2.54mm:PinHeader_1x05_P2.54mm_Vertical
- J110: footprint (none) -> Connector_PinHeader_2.54mm:PinHeader_1x04_P2.54mm_Vertical
- J111: footprint (none) -> Connector_PinSocket_2.54mm:PinSocket_2x22_P2.54mm_Vertical
- R101, R102: footprint (none) -> Resistor_SMD:R_0805_2012Metric_Pad1.15x1.40mm_HandSolder
- TP104, TP105: footprint (none) -> Connector_PinHeader_2.54mm:PinHeader_1x01_P2.54mm_Vertical
- U101: footprint TO_SOT_Packages_SMD:SOT-223 -> Package_TO_SOT_SMD:SOT-223
Changed lines of the file:
@@
 F 0 "U101" H 6400 1515 50  0000 C CNN
 F 1 "AP7361C-33" H 6400 1424 50  0000 C CNN
-F 2 "TO_SOT_Packages_SMD:SOT-223" H 6500 1500 50  0001 C CNN
+F 2 "Package_TO_SOT_SMD:SOT-223" H 6500 1500 50  0001 C CNN
 F 3 "https://www.diodes.com/assets/Datasheets/AP7361C.pdf" H 6400 1300 50  0001 C CNN
 	1    6400 1250
@@
 F 0 "C102" H 5700 1650 50  0000 L CNN
 F 1 "100n" H 5700 1450 50  0000 L CNN
-F 2 "" H 5688 1400 50  0001 C CNN
+F 2 "Capacitor_SMD:C_0805_2012Metric_Pad1.15x1.40mm_HandSolder" H 5688 1400 50  0001 C CNN
 F 3 "" H 5650 1550 50  0001 C CNN
 	1    5650 1550
@@
 F 0 "C104" H 7250 1650 50  0000 L CNN
 F 1 "4u7" H 7250 1450 50  0000 L CNN
-F 2 "" H 7238 1400 50  0001 C CNN
+F 2 "Capacitor_SMD:C_0805_2012Metric_Pad1.15x1.40mm_HandSolder" H 7238 1400 50  0001 C CNN
 F 3 "" H 7200 1550 50  0001 C CNN
 	1    7200 1550
@@
 F 0 "C105" H 7650 1650 50  0000 L CNN
 F 1 "10u" H 7650 1450 50  0000 L CNN
-F 2 "" H 7638 1400 50  0001 C CNN
+F 2 "Capacitor_SMD:C_0805_2012Metric_Pad1.15x1.40mm_HandSolder" H 7638 1400 50  0001 C CNN
 F 3 "" H 7600 1550 50  0001 C CNN
 	1    7600 1550
@@
 F 0 "C101" H 5300 1650 50  0000 L CNN
 F 1 "4u7" H 5300 1450 50  0000 L CNN
-F 2 "" H 5288 1400 50  0001 C CNN
+F 2 "Capacitor_SMD:C_0805_2012Metric_Pad1.15x1.40mm_HandSolder" H 5288 1400 50  0001 C CNN
 F 3 "" H 5250 1550 50  0001 C CNN
 	1    5250 1550
@@
 F 0 "J101" H 800 2600 50  0000 C CNN
 F 1 "CAN" H 800 2050 50  0000 C CNN
-F 2 "" H 800 2350 50  0001 C CNN
+F 2 "supermileage_footprints:Molex-duraClick-4conn" H 800 2350 50  0001 C CNN
 F 3 "~" H 800 2350 50  0001 C CNN
 	1    800  2350
@@
 F 0 "J102" H 800 3800 50  0000 C CNN
 F 1 "Throttle" H 800 3200 50  0000 C CNN
-F 2 "" H 800 3550 50  0001 C CNN
+F 2 "supermileage_footprints:Molex-duraClick-4conn" H 800 3550 50  0001 C CNN
 F 3 "~" H 800 3550 50  0001 C CNN
 	1    800  3550
@@
 F 0 "R101" H 2450 4700 50  0000 L CNN
 F 1 "10K" H 2450 4550 50  0000 L CNN
-F 2 "" V 2580 4550 50  0001 C CNN
+F 2 "Resistor_SMD:R_0805_2012Metric_Pad1.15x1.40mm_HandSolder" V 2580 4550 50  0001 C CNN
 F 3 "" H 2650 4550 50  0001 C CNN
 	1    2650 4550
@@
 F 0 "J111" H 9275 833 50  0000 C CNN
 F 1 "Trinamic-Bridge" H 9275 924 50  0000 C CNN
-F 2 "" H 8750 2150 50  0001 C CNN
+F 2 "Connector_PinSocket_2.54mm:PinSocket_2x22_P2.54mm_Vertical" H 8750 2150 50  0001 C CNN
 F 3 "" H 8750 2150 50  0001 C CNN
 	1    9250 2150
@@
 F 0 "R102" H 2150 2400 50  0000 L CNN
 F 1 "10K" H 2200 2300 50  0000 L CNN
-F 2 "" V 2380 2350 50  0001 C CNN
+F 2 "Resistor_SMD:R_0805_2012Metric_Pad1.15x1.40mm_HandSolder" V 2380 2350 50  0001 C CNN
 F 3 "~" H 2450 2350 50  0001 C CNN
 	1    2450 2350
@@
 F 0 "J108" V 5200 3550 50  0000 C CNN
 F 1 "CAN_DBG" V 5300 3750 50  0000 C CNN
-F 2 "" H 5200 3800 50  0001 C CNN
+F 2 "Connector_PinHeader_2.54mm:PinHeader_1x02_P2.54mm_Vertical" H 5200 3800 50  0001 C CNN
 F 3 "~" H 5200 3800 50  0001 C CNN
 	1    5200 3800
@@
 F 0 "J110" V 7850 3450 50  0000 C CNN
 F 1 "SPI_DBG" V 7950 3750 50  0000 C CNN
-F 2 "" H 7850 3800 50  0001 C CNN
+F 2 "Connector_PinHeader_2.54mm:PinHeader_1x04_P2.54mm_Vertical" H 7850 3800 50  0001 C CNN
 F 3 "~" H 7850 3800 50  0001 C CNN
 	1    7850 3800
@@
 F 0 "J109" H 2100 3900 50  0000 C CNN
 F 1 "ABN Encoder" V 2200 3550 50  0000 C CNN
-F 2 "" H 2100 3550 50  0001 C CNN
+F 2 "Connector_PinHeader_2.54mm:PinHeader_1x05_P2.54mm_Vertical" H 2100 3550 50  0001 C CNN
 F 3 "~" H 2100 3550 50  0001 C CNN
 	1    2100 3550
@@
 F 0 "TP102" H 1200 7250 50  0000 L CNN
 F 1 "5v_TP" H 1150 7350 50  0000 L CNN
-F 2 "" H 1250 7450 50  0001 C CNN
+F 2 "Connector_PinHeader_2.54mm:PinHeader_1x02_P2.54mm_Vertical" H 1250 7450 50  0001 C CNN
 F 3 "~" H 1250 7450 50  0001 C CNN
 	1    1250 7450
@@
 F 0 "TP103" H 1550 7250 50  0000 L CNN
 F 1 "3v3_TP" H 1500 7350 50  0000 L CNN
-F 2 "" H 1600 7450 50  0001 C CNN
+F 2 "Connector_PinHeader_2.54mm:PinHeader_1x02_P2.54mm_Vertical" H 1600 7450 50  0001 C CNN
 F 3 "~" H 1600 7450 50  0001 C CNN
 	1    1600 7450
@@
 F 0 "TP104" H 2008 7770 50  0000 L CNN
 F 1 "GND_TP" H 1800 7900 50  0000 L CNN
-F 2 "" H 2150 7650 50  0001 C CNN
+F 2 "Connector_PinHeader_2.54mm:PinHeader_1x01_P2.54mm_Vertical" H 2150 7650 50  0001 C CNN
 F 3 "~" H 2150 7650 50  0001 C CNN
 	1    1950 7650
@@
 F 0 "TP105" H 2358 7770 50  0000 L CNN
 F 1 "GND_TP" H 2200 7900 50  0000 L CNN
-F 2 "" H 2500 7650 50  0001 C CNN
+F 2 "Connector_PinHeader_2.54mm:PinHeader_1x01_P2.54mm_Vertical" H 2500 7650 50  0001 C CNN
 F 3 "~" H 2500 7650 50  0001 C CNN
 	1    2300 7650
@@
 F 0 "TP101" H 850 7250 50  0000 L CNN
 F 1 "5v_TP" H 800 7350 50  0000 L CNN
-F 2 "" H 900 7450 50  0001 C CNN
+F 2 "Connector_PinHeader_2.54mm:PinHeader_1x02_P2.54mm_Vertical" H 900 7450 50  0001 C CNN
 F 3 "~" H 900 7450 50  0001 C CNN
 	1    900  7450
