File: motor-controller-hw/power-supply.sch (KiCad schematic (older format))
At the start: 0 parts

Commit message: Added more signals to the top level diagram
Parts:
- added JP?: GND_Tie, symbol Device:Jumper_NC_Small
Connections:
- net labels added: 3.6v, 5.0v, BatCurrent, BatVoltage, D_GND, GNDD, GNDPWR, P_GND, vBat
- wire segments 0 -> 8
Other:
- note added: "Seprate grounds for digital supply \nand power, joined with a tie so seprate \nnets are generated on the PCB."
Changed lines of the file:
@@
 $Descr A4 11693 8268
 encoding utf-8
-Sheet 1 7
+Sheet 5 7
 Title ""
 Date ""
@@
 Comment4 ""
 $EndDescr
+Text HLabel 9900 1850 2    50   Input ~ 0
+BatVoltage
+Text HLabel 9900 1950 2    50   Input ~ 0
+BatCurrent
+Text HLabel 9900 1700 2    50   Output ~ 0
+3.6v
+Text HLabel 9900 1600 2    50   Output ~ 0
+5.0v
+Text HLabel 9900 1500 2    50   Output ~ 0
+vBat
+Text HLabel 9900 2300 2    50   UnSpc ~ 0
+D_GND
+Text HLabel 9900 2400 2    50   UnSpc ~ 0
+P_GND
+$Comp
+L power:GNDPWR #PWR?
+U 1 1 5BBC9D0F
+P 9650 2500
+AR Path="/5BAADA79/5BBC9D0F" Ref="#PWR?"  Part="1"
+AR Path="/5BAADA7C/5BBC9D0F" Ref="#PWR?"  Part="1"
+F 0 "#PWR?" H 9650 2300 50  0001 C CNN
+F 1 "GNDPWR" H 9654 2346 50  0000 C CNN
+F 2 "" H 9650 2450 50  0001 C CNN
+F 3 "" H 9650 2450 50  0001 C CNN
+	1    9650 2500
+	-1   0    0    -1
+$EndComp
+$Comp
+L power:GNDD #PWR?
+U 1 1 5BBC9D15
+P 9350 2500
+AR Path="/5BAADA79/5BBC9D15" Ref="#PWR?"  Part="1"
+AR Path="/5BAADA7C/5BBC9D15" Ref="#PWR?"  Part="1"
+F 0 "#PWR?" H 9350 2250 50  0001 C CNN
+F 1 "GNDD" H 9354 2345 50  0000 C CNN
+F 2 "" H 9350 2500 50  0001 C CNN
+F 3 "" H 9350 2500 50  0001 C CNN
+	1    9350 2500
+	-1   0    0    -1
+$EndComp
+Wire Wire Line
+	9900 2300 9350 2300
+Wire Wire Line
+	9350 2300 9350 2500
+Wire Wire Line
+	9900 2400 9650 2400
+Wire Wire Line
+	9650 2400 9650 2500
+Text Notes 9000 3100 0    50   ~ 0
+Seprate grounds for digital supply \nand power, joined with a tie so seprate \nnets are generated on the PCB.
+$Comp
+L Device:Jumper_NC_Small JP?
+U 1 1 5BBC9DC6
+P 9550 3400
+F 0 "JP?" H 9550 3612 50  0000 C CNN
+F 1 "GND_Tie" H 9550 3521 50  0000 C CNN
+F 2 "" H 9550 3400 50  0001 C CNN
+F 3 "~" H 9550 3400 50  0001 C CNN
+	1    9550 3400
+	1    0    0    -1
+$EndComp
+$Comp
+L power:GNDD #PWR?
+U 1 1 5BBC9E50
+P 9400 3450
+AR Path="/5BAADA79/5BBC9E50" Ref="#PWR?"  Part="1"
+AR Path="/5BAADA7C/5BBC9E50" Ref="#PWR?"  Part="1"
+F 0 "#PWR?" H 9400 3200 50  0001 C CNN
+F 1 "GNDD" H 9404 3295 50  0000 C CNN
+F 2 "" H 9400 3450 50  0001 C CNN
+F 3 "" H 9400 3450 50  0001 C CNN
+	1    9400 3450
+	-1   0    0    -1
+$EndComp
+$Comp
+L power:GNDPWR #PWR?
+U 1 1 5BBC9E5D
+P 9700 3450
+AR Path="/5BAADA79/5BBC9E5D" Ref="#PWR?"  Part="1"
+AR Path="/5BAADA7C/5BBC9E5D" Ref="#PWR?"  Part="1"
+F 0 "#PWR?" H 9700 3250 50  0001 C CNN
+F 1 "GNDPWR" H 9704 3296 50  0000 C CNN
+F 2 "" H 9700 3400 50  0001 C CNN
+F 3 "" H 9700 3400 50  0001 C CNN
+	1    9700 3450
+	-1   0    0    -1
+$EndComp
+Wire Wire Line
+	9400 3450 9400 3400
+Wire Wire Line
+	9400 3400 9450 3400
+Wire Wire Line
+	9650 3400 9700 3400
+Wire Wire Line
+	9700 3400 9700 3450
 $EndSCHEMATC

Commit message: Changed hierarchy Added input protection circuitry
Connections:
- net labels added: 3.3v
- net labels removed: 3.6v, BatCurrent, BatVoltage
Changed lines of the file:
@@
 $Descr A4 11693 8268
 encoding utf-8
-Sheet 5 7
+Sheet 4 5
 Title ""
 Date ""
 Rev ""
-Comp ""
+Comp "Cedarville University"
 Comment1 ""
 Comment2 ""
@@
 Comment4 ""
 $EndDescr
-Text HLabel 9900 1850 2    50   Input ~ 0
-BatVoltage
-Text HLabel 9900 1950 2    50   Input ~ 0
-BatCurrent
 Text HLabel 9900 1700 2    50   Output ~ 0
-3.6v
+3.3v
 Text HLabel 9900 1600 2    50   Output ~ 0
 5.0v

Commit message: Finished Input Protection Added annotations to the title block
Parts:
- gave numbers to parts that had none: 1
Changed lines of the file:
@@
 Rev ""
 Comp "Cedarville University"
-Comment1 ""
-Comment2 ""
-Comment3 ""
+Comment1 "Supermileage Motor Controller"
+Comment2 "Senior Design 2018-2019"
+Comment3 "Samuel Ellicott"
 Comment4 ""
 $EndDescr
@@
 P 9650 2500
 AR Path="/5BAADA79/5BBC9D0F" Ref="#PWR?"  Part="1"
-AR Path="/5BAADA7C/5BBC9D0F" Ref="#PWR?"  Part="1"
-F 0 "#PWR?" H 9650 2300 50  0001 C CNN
+AR Path="/5BAADA7C/5BBC9D0F" Ref="#PWR0403"  Part="1"
+F 0 "#PWR0403" H 9650 2300 50  0001 C CNN
 F 1 "GNDPWR" H 9654 2346 50  0000 C CNN
 F 2 "" H 9650 2450 50  0001 C CNN
@@
 P 9350 2500
 AR Path="/5BAADA79/5BBC9D15" Ref="#PWR?"  Part="1"
-AR Path="/5BAADA7C/5BBC9D15" Ref="#PWR?"  Part="1"
-F 0 "#PWR?" H 9350 2250 50  0001 C CNN
+AR Path="/5BAADA7C/5BBC9D15" Ref="#PWR0401"  Part="1"
+F 0 "#PWR0401" H 9350 2250 50  0001 C CNN
 F 1 "GNDD" H 9354 2345 50  0000 C CNN
 F 2 "" H 9350 2500 50  0001 C CNN
@@
 Seprate grounds for digital supply \nand power, joined with a tie so seprate \nnets are generated on the PCB.
 $Comp
-L Device:Jumper_NC_Small JP?
+L Device:Jumper_NC_Small JP401
 U 1 1 5BBC9DC6
 P 9550 3400
-F 0 "JP?" H 9550 3612 50  0000 C CNN
+F 0 "JP401" H 9550 3612 50  0000 C CNN
 F 1 "GND_Tie" H 9550 3521 50  0000 C CNN
 F 2 "" H 9550 3400 50  0001 C CNN
@@
 P 9400 3450
 AR Path="/5BAADA79/5BBC9E50" Ref="#PWR?"  Part="1"
-AR Path="/5BAADA7C/5BBC9E50" Ref="#PWR?"  Part="1"
-F 0 "#PWR?" H 9400 3200 50  0001 C CNN
+AR Path="/5BAADA7C/5BBC9E50" Ref="#PWR0402"  Part="1"
+F 0 "#PWR0402" H 9400 3200 50  0001 C CNN
 F 1 "GNDD" H 9404 3295 50  0000 C CNN
 F 2 "" H 9400 3450 50  0001 C CNN
@@
 P 9700 3450
 AR Path="/5BAADA79/5BBC9E5D" Ref="#PWR?"  Part="1"
-AR Path="/5BAADA7C/5BBC9E5D" Ref="#PWR?"  Part="1"
-F 0 "#PWR?" H 9700 3250 50  0001 C CNN
+AR Path="/5BAADA7C/5BBC9E5D" Ref="#PWR0404"  Part="1"
+F 0 "#PWR0404" H 9700 3250 50  0001 C CNN
 F 1 "GNDPWR" H 9704 3296 50  0000 C CNN
 F 2 "" H 9700 3400 50  0001 C CNN

Commit message: Added system library parts to project library Added a few more comments to IO.sch Added TMC4671 SPI bus as an output for microcontroller.sch Added some connections in the overview page Updated schematic dates
Parts:
- JP401: symbol Device:Jumper_NC_Small -> MotorControllerParts:Jumper_NC_Small
Changed lines of the file:
@@
 Seprate grounds for digital supply \nand power, joined with a tie so seprate \nnets are generated on the PCB.
 $Comp
-L Device:Jumper_NC_Small JP401
+L MotorControllerParts:Jumper_NC_Small JP401
 U 1 1 5BBC9DC6
 P 9550 3400

Commit message: power-supply.sch: Added some voltage regulators removed from main schematic
Parts:
- added C?: 100n, symbol MotorControllerParts:C
- added C? (x2): 4u7, symbol MotorControllerParts:C
- added C?: 10u, symbol MotorControllerParts:C
- added C?: 33u, symbol MotorControllerParts:C
- added D?: 18V Zener, symbol Device:D_Zener_ALT
- added Q?: Q_PMOS_GDS, symbol Device:Q_PMOS_GDS
- added R?: 10K, symbol MotorControllerParts:R
- added U?: D36V6F5, supermileage_footprints:D36V6Fx, symbol MotorControllerParts:D36V6Fx
- added U?: AP7361C-33, TO_SOT_Packages_SMD:SOT-223, symbol MotorControllerParts:AP7361C
Connections:
- net labels added: +3.3V, +5V, +BATT, VBatt, Vin
- net labels removed: vBat
- wire segments 8 -> 53
- no-connect marks 0 -> 1
Other:
- note added: "3.3V linear voltage regulator for the low voltage electronics. The selected\nregulator can supply 1A of output current, which is more than what the 5V \nswitching regulator can supply. The 4.7uF output capacitor should have a \nfairly low ESR."
- note added: "5V switching regulator, up to 50V input, maximum 600mA output current. \nP-Channel MOSFET for an ideal diode with a 18v zener diode to protect the \nMOSFET gate. The 10K resistor limits the zener diode current to 3mA at \n48V input."
