File: motor-controller-hw/TMC4671.sch (KiCad schematic (older format))
At the start: 0 parts

Commit message: TMC4671.sch: added a decoupling capacitors other base components
Parts:
- added C? (x10): 100n, symbol MotorControllerParts:C
- added C? (x2): 4u7, symbol MotorControllerParts:C
- added C?: 470n, symbol MotorControllerParts:C
- added J?: User USART, symbol MotorControllerParts:Conn_01x03
- added R? (x2): 20K, symbol MotorControllerParts:R
- added R? (x2): 10K, symbol MotorControllerParts:R
- added U?: TMC4671, symbol MotorControllerParts:TMC4671
Connections:
- net labels added: +3.3V, +5V, 1v8, A_Current, B_Current, GNDD, HALL_A, HALL_B, HALL_C, PWM_AH, PWM_AL, PWM_BH, PWM_BL, PWM_CH, PWM_CL, PWM_Phase_AH, PWM_Phase_AL, PWM_Phase_BH, PWM_Phase_BL, PWM_Phase_CH, PWM_Phase_CL, Phase_A_Current, Phase_B_Current, SPI_CS, SPI_MISO, SPI_MOSI, SPI_SCK, USART_Rx, USART_Tx, ~SPI_CS
- wire segments 0 -> 143
- no-connect marks 0 -> 14

Commit message: Moving away from TMC4671
Parts:
- added C? (x2): 100n, symbol MotorControllerParts:C
- added C? (x2): 100p, symbol MotorControllerParts:C
- added C?: 10n, symbol MotorControllerParts:C
- added R? (x3): 10K, symbol MotorControllerParts:R
- added R?: 110K, symbol MotorControllerParts:R
- added R? (x2): 100R, symbol MotorControllerParts:R
- added X?: IQXO-50, Oscillator:Oscillator_SMD_IQD_IQXO70-4Pin_7.5x5.0mm, symbol MotorControllerParts:IQXO-50
Connections:
- net labels added: +BATT, Batt_Current, Batt_V, CLK, DGND, ENC_A, ENC_B, ENC_N, En_In, En_Out, PWM_DH, PWM_DL, PWM_Idle_H, PWM_Idle_L, PWM_Phase_DH, PWM_Phase_DL, Status, VBatt
- wire segments 143 -> 198
- no-connect marks 14 -> 19

Commit message: Voltage regualtor changes, name changes, and HANDS!!!
Parts:
- removed C?: 100p, symbol MotorControllerParts:C
- removed C?: 100n, symbol MotorControllerParts:C
- removed R?: 100R, symbol MotorControllerParts:R
- added C? (x2): 100n, symbol MotorControllerParts:C
- added J?: Trinamic_TRMI, symbol MotorControllerParts:Trinamic_TRMI
- added R?: 100R, symbol MotorControllerParts:R
- added TP? (x11): TestPoint, symbol MotorControllerParts:TestPoint
- added TP?: A_I_TP, symbol MotorControllerParts:TestPoint_2Pole
- added TP?: B_I_TP, symbol MotorControllerParts:TestPoint_2Pole
- added TP?: Batt_I_TP, symbol MotorControllerParts:TestPoint_2Pole
- added TP?: Batt_V_TP, symbol MotorControllerParts:TestPoint_2Pole
- C?: value 100p -> 100n
- J?: value User USART -> TMC4671 USART
Connections:
- net labels added: Brake, Brake_Chopper, RTMI_CS, RTMI_MISO, RTMI_MOSI, RTMI_SCK, RTMI_TRG
- net labels removed: +BATT
- wire segments 198 -> 254
- no-connect marks 19 -> 8
Other:
- note added: "Battery Voltage and Current\nCurrent RC filter set for 1.59KHz\nVoltage RC filter set for 1.59KHz"
- note added: "Phase current low pass filters\n RC constant set for 15KHz"

Commit message: Working schematics
Parts:
- added C? (x2): 100n, symbol MotorControllerParts:C
- added TP? (x5): TestPoint, symbol MotorControllerParts:TestPoint
- added TP?: B_Ref, symbol MotorControllerParts:TestPoint
- added TP?: A_Ref, symbol MotorControllerParts:TestPoint
- R? (x2): value 20K -> 10K
Connections:
- net labels added: A_Current_Ref, B_Current_Ref
- wire segments 254 -> 269
- no-connect marks 8 -> 3
Other:
- note added: "Decoupling capacitors"
- note added: "TMC4671 Clock Chip"
- note added: "TMC4671 Debug interfaces"
- note added: "Voltage references for the current measurement ADC's"

Commit message: Compacted schematic layout
Parts:
- gave numbers to parts that had none: 56

Commit message: Added footprints, changed pdf
Parts:
- C401, C402, C403, C404, C405, C406, C407, C408, C409, C410, C411, C412, C413, C414, C415, C416, C417, C418, C419, C420: footprint (none) -> Capacitor_SMD:C_0805_2012Metric_Pad1.15x1.40mm_HandSolder
- J402, TP401, TP402: footprint (none) -> Connector_PinHeader_2.54mm:PinHeader_1x03_P2.54mm_Vertical
- R401, R402, R403, R404, R405, R406, R407, R408, R409, R410: footprint (none) -> Resistor_SMD:R_0805_2012Metric_Pad1.15x1.40mm_HandSolder
- TP403, TP404, TP405, TP406, TP407, TP408, TP409, TP410, TP411, TP412, TP413, TP414, TP415, TP416, TP417, TP418: footprint (none) -> TestPoint:TestPoint_Pad_D1.0mm
- TP419, TP420, TP421, TP422: footprint (none) -> Connector_PinHeader_2.54mm:PinHeader_1x02_P2.54mm_Vertical
- U401: footprint (none) -> supermileage_footprints:TMC4671
