File: motor-controller-hw/IO.sch (KiCad schematic (older format))
At the start: 32 parts, among them U501 MCP6004, U502 MCP6004, U503 MCP6004, U504 74HC14, U505 74HC244, U506 mcp2562

Commit message: Moving away from TMC4671
Parts:
- removed C514: 100n, symbol MotorControllerParts:C
- removed JP501: HALL Select, symbol MotorControllerParts:Conn_02x02_Odd_Even
- removed R507, R509: 10K, symbol MotorControllerParts:R
- removed U504: 74HC14, symbol 74xx:74HC14
- removed U505: 74HC244, symbol 74xx:74HC244
- added C511: 100n, symbol MotorControllerParts:C
- added C? (x3): 100p, symbol MotorControllerParts:C
- added R? (x3): 22R, symbol MotorControllerParts:R
- added R? (x3): 4K7, symbol MotorControllerParts:R
- added U504, U? (x7): 74HC7014, Package_SO:SOIC-14_3.9x8.7mm_P1.27mm, symbol 74xx:74HC7014
- renumbered C511 to C512, C512 to C514
Connections:
- net labels added: A_HALL_TVS, B_HALL_TVS, Phase_A_ABN_i, Phase_B_ABN_i, Phase_N_ABN_i
- net labels removed: Phase_A_HALL_FX_i, Phase_A_HAL_FX_i, Phase_B_HALL_FX_i, Phase_B_HAL_FX_i, Phase_C_HALL_FX_i, Phase_C_HAL_FX_i, Serial_Rx, Serial_Tx, TMC4671_RX, TMC4671_Rx_i, TMC4671_TX, TMC4671_Tx_i
- wire segments 277 -> 263
- no-connect marks 2 -> 0
Other:
- note added: "Hall Input Filtering"
- note removed: "Hall Input Select"

Commit message: Added scmitt triggers to the input protection circuitry
Parts:
- removed U? (x2): 74HC7014, Package_SO:SOIC-14_3.9x8.7mm_P1.27mm, symbol 74xx:74HC7014
- added C? (x3): 100p, symbol MotorControllerParts:C
- added R? (x3): 22R, symbol MotorControllerParts:R
- added R? (x3): 4K7, symbol MotorControllerParts:R
- added U? (x5): 74HC7014, Package_SO:SOIC-14_3.9x8.7mm_P1.27mm, symbol 74xx:74HC7014
Connections:
- net labels added: A_ABN, A_ABN_TVS, A_ABN_i, B_ABN, B_ABN_TVS, B_ABN_i, N_ABN, N_ABN_TVS, N_ABN_i
- net labels removed: Phase_A_ABN_i, Phase_B_ABN_i, Phase_N_ABN_i
- wire segments 263 -> 287

Commit message: Voltage regualtor changes, name changes, and HANDS!!!
Parts:
- removed R? (x4): 22R, symbol MotorControllerParts:R
- removed U? (x3): 74HC7014, Package_SO:SOIC-14_3.9x8.7mm_P1.27mm, symbol 74xx:74HC7014
- added R? (x4): 100R, symbol MotorControllerParts:R
- C? (x6): value 100p -> 100n
- R? (x2): value 22R -> 100R
Connections:
- net labels added: ENC_A, ENC_A_i, ENC_B, ENC_B_i, ENC_N, ENC_N_i
- net labels removed: A_ABN, A_ABN_i, B_ABN, B_ABN_i, N_ABN, N_ABN_i
Other:
- note added: "ABN Encoder Input Filtering"
- note added: "Lowpass filters set for about 1.59Khz\nSchmitt trigger inputs for taking out noise"
- note added: "Lowpass filters set for about 72Khz\nSchmitt trigger inputs for taking out noise"
Changed lines of the file:
@@
 $Descr USLedger 17000 11000
 encoding utf-8
-Sheet 4 4
+Sheet 3 4
 Title "Input Protection and Filtering"
 Date "2018-11-17"
@@
 Hall Input Filtering
 Text HLabel 1350 7050 0    50   Input ~ 0
-A_ABN_i
+ENC_A_i
 Text HLabel 1350 7150 0    50   Input ~ 0
-B_ABN_i
+ENC_B_i
 Text HLabel 1350 7250 0    50   Input ~ 0
-N_ABN_i
-Text Label 1750 7050 2    50   ~ 0
-A_ABN_i
-Text Label 1750 7150 2    50   ~ 0
-B_ABN_i
-Text Label 1750 7250 2    50   ~ 0
-N_ABN_i
+ENC_N_i
 Wire Wire Line
 	1350 7050 1750 7050
@@
 Wire Wire Line
 	15200 4050 15650 4050
-Text Notes 19400 1050 0    59   ~ 0
+Text Notes 13000 8850 0    59   ~ 0
 This sheet contains input/output proteciton and conditioning circuitry. \nNote that the TMC4671 and stm32 USB lines pass through this sheet\nwithout modification.
 Text Label 10800 6400 2    50   ~ 0
@@
 L 74xx:74HC7014 U?
 U 4 1 5CCC2417
-P 20800 4150
-F 0 "U?" H 20800 4467 50  0000 C CNN
-F 1 "74HC7014" H 20800 4376 50  0000 C CNN
-F 2 "Package_SO:SOIC-14_3.9x8.7mm_P1.27mm" H 20800 4150 50  0001 C CNN
-F 3 "https://assets.nexperia.com/documents/data-sheet/74HC7014.pdf" H 20800 4150 50  0001 C CNN
-	4    20800 4150
+P 13550 3900
+F 0 "U?" H 13550 4217 50  0000 C CNN
+F 1 "74HC7014" H 13550 4126 50  0000 C CNN
+F 2 "Package_SO:SOIC-14_3.9x8.7mm_P1.27mm" H 13550 3900 50  0001 C CNN
+F 3 "https://assets.nexperia.com/documents/data-sheet/74HC7014.pdf" H 13550 3900 50  0001 C CNN
+	4    13550 3900
 	1    0    0    -1
 $EndComp
@@
 L 74xx:74HC7014 U?
 U 5 1 5CCC25DA
-P 20800 4650
-F 0 "U?" H 20800 4967 50  0000 C CNN
-F 1 "74HC7014" H 20800 4876 50  0000 C CNN
-F 2 "Package_SO:SOIC-14_3.9x8.7mm_P1.27mm" H 20800 4650 50  0001 C CNN
-F 3 "https://assets.nexperia.com/documents/data-sheet/74HC7014.pdf" H 20800 4650 50  0001 C CNN
-	5    20800 4650
+P 13550 5150
+F 0 "U?" H 13550 5467 50  0000 C CNN
+F 1 "74HC7014" H 13550 5376 50  0000 C CNN
+F 2 "Package_SO:SOIC-14_3.9x8.7mm_P1.27mm" H 13550 5150 50  0001 C CNN
+F 3 "https://assets.nexperia.com/documents/data-sheet/74HC7014.pdf" H 13550 5150 50  0001 C CNN
+	5    13550 5150
 	1    0    0    -1
 $EndComp
@@
 L 74xx:74HC7014 U?
 U 6 1 5CCC272E
-P 20800 5250
-F 0 "U?" H 20800 5567 50  0000 C CNN
-F 1 "74HC7014" H 20800 5476 50  0000 C CNN
-F 2 "Package_SO:SOIC-14_3.9x8.7mm_P1.27mm" H 20800 5250 50  0001 C CNN
-F 3 "https://assets.nexperia.com/documents/data-sheet/74HC7014.pdf" H 20800 5250 50  0001 C CNN
-	6    20800 5250
+P 13550 6400
+F 0 "U?" H 13550 6717 50  0000 C CNN
+F 1 "74HC7014" H 13550 6626 50  0000 C CNN
+F 2 "Package_SO:SOIC-14_3.9x8.7mm_P1.27mm" H 13550 6400 50  0001 C CNN
+F 3 "https://assets.nexperia.com/documents/data-sheet/74HC7014.pdf" H 13550 6400 50  0001 C CNN
+	6    13550 6400
 	1    0    0    -1
 $EndComp
@@
 $Comp
 L MotorControllerParts:R R?
-U 1 1 5CD97073
-P 8600 3900
-F 0 "R?" V 8500 3850 50  0000 L CNN
-F 1 "22R" V 8700 3850 50  0000 L CNN
-F 2 "" V 8530 3900 50  0001 C CNN
-F 3 "~" H 8600 3900 50  0001 C CNN
-	1    8600 3900
-	0    1    1    0
-$EndComp
-$Comp
-L MotorControllerParts:R R?
 U 1 1 5CE69E61
 P 9000 3700
@@
 P 9000 4100
 F 0 "C?" H 9115 4146 50  0000 L CNN
-F 1 "100p" H 9115 4055 50  0000 L CNN
+F 1 "100n" H 9115 4055 50  0000 L CNN
 F 2 "" H 9038 3950 50  0001 C CNN
 F 3 "~" H 9000 4100 50  0001 C CNN
@@
 $Comp
 L MotorControllerParts:R R?
-U 1 1 5CF745B8
-P 8600 5150
-F 0 "R?" V 8500 5100 50  0000 L CNN
-F 1 "22R" V 8700 5100 50  0000 L CNN
-F 2 "" V 8530 5150 50  0001 C CNN
-F 3 "~" H 8600 5150 50  0001 C CNN
-	1    8600 5150
-	0    1    1    0
-$EndComp
-$Comp
-L MotorControllerParts:R R?
 U 1 1 5CF745BF
 P 9000 4950
@@
 P 9000 5350
 F 0 "C?" H 9115 5396 50  0000 L CNN
-F 1 "100p" H 9115 5305 50  0000 L CNN
+F 1 "100n" H 9115 5305 50  0000 L CNN
 F 2 "" H 9038 5200 50  0001 C CNN
 F 3 "~" H 9000 5350 50  0001 C CNN
@@
 $Comp
 L MotorControllerParts:R R?
-U 1 1 5D0817B7
-P 8600 6400
-F 0 "R?" V 8500 6350 50  0000 L CNN
-F 1 "22R" V 8700 6350 50  0000 L CNN
-F 2 "" V 8530 6400 50  0001 C CNN
-F 3 "~" H 8600 6400 50  0001 C CNN
-	1    8600 6400
-	0    1    1    0
-$EndComp
-$Comp
-L MotorControllerParts:R R?
 U 1 1 5D0817BE
 P 9000 6200
@@
 P 9000 6600
 F 0 "C?" H 9115 6646 50  0000 L CNN
-F 1 "100p" H 9115 6555 50  0000 L CNN
+F 1 "100n" H 9115 6555 50  0000 L CNN
 F 2 "" H 9038 6450 50  0001 C CNN
 F 3 "~" H 9000 6600 50  0001 C CNN
@@
 Wire Notes Line
 	11200 7200 11200 3100
-Text Notes 12700 3200 0    50   ~ 0
-Hall Input Filtering
-Text Label 14400 6400 2    50   ~ 0
-Phase_C_HALL
-Text Label 14400 5150 2    50   ~ 0
-Phase_B_HALL
-Text Label 14400 3900 2    50   ~ 0
-Phase_A_HALL
-$Comp
-L 74xx:74HC7014 U?
-U 1 1 5C097299
-P 13550 3900
-F 0 "U?" H 13550 4217 50  0000 C CNN
-F 1 "74HC7014" H 13550 4126 50  0000 C CNN
-F 2 "Package_SO:SOIC-14_3.9x8.7mm_P1.27mm" H 13550 3900 50  0001 C CNN
-F 3 "https://assets.nexperia.com/documents/data-sheet/74HC7014.pdf" H 13550 3900 50  0001 C CNN
-	1    13550 3900
-	1    0    0    -1
-$EndComp
+Text Notes 12400 3200 0    50   ~ 0
+ABN Encoder Input Filtering
 $Comp
 L MotorControllerParts:R R?
@@
 P 12200 3900
 F 0 "R?" V 12100 3850 50  0000 L CNN
-F 1 "22R" V 12300 3850 50  0000 L CNN
+F 1 "100R" V 12300 3800 50  0000 L CNN
 F 2 "" V 12130 3900 50  0001 C CNN
 F 3 "~" H 12200 3900 50  0001 C CNN
@@
 P 12600 4100
 F 0 "C?" H 12715 4146 50  0000 L CNN
-F 1 "100p" H 12715 4055 50  0000 L CNN
+F 1 "100n" H 12715 4055 50  0000 L CNN
 F 2 "" H 12638 3950 50  0001 C CNN
 F 3 "~" H 12600 4100 50  0001 C CNN
@@
 	12600 3900 13250 3900
 Wire Wire Line
-	13850 3900 14400 3900
+	13850 3900 14200 3900
 Wire Wire Line
 	12600 4300 12600 4250
@@
 P 12200 5150
 F 0 "R?" V 12100 5100 50  0000 L CNN
-F 1 "22R" V 12300 5100 50  0000 L CNN
+F 1 "100R" V 12300 5050 50  0000 L CNN
 F 2 "" V 12130 5150 50  0001 C CNN
 F 3 "~" H 12200 5150 50  0001 C CNN
@@
 P 12600 5350
 F 0 "C?" H 12715 5396 50  0000 L CNN
-F 1 "100p" H 12715 5305 50  0000 L CNN
+F 1 "100n" H 12715 5305 50  0000 L CNN
 F 2 "" H 12638 5200 50  0001 C CNN
 F 3 "~" H 12600 5350 50  0001 C CNN
@@
 	12600 5550 12600 5500
 Wire Wire Line
-	14400 5150 13850 5150
+	14200 5150 13850 5150
 $Comp
 L MotorControllerParts:GNDD #PWR?
@@
 $Comp
 L MotorControllerParts:R R?
-U 1 1 5C0972F4
-P 12200 6400
-F 0 "R?" V 12100 6350 50  0000 L CNN
-F 1 "22R" V 12300 6350 50  0000 L CNN
-F 2 "" V 12130 6400 50  0001 C CNN
-F 3 "~" H 12200 6400 50  0001 C CNN
-	1    12200 6400
-	0    1    1    0
-$EndComp
-$Comp
-L MotorControllerParts:R R?
 U 1 1 5C0972FB
 P 12600 6200
@@
 P 12600 6600
 F 0 "C?" H 12715 6646 50  0000 L CNN
-F 1 "100p" H 12715 6555 50  0000 L CNN
+F 1 "100n" H 12715 6555 50  0000 L CNN
 F 2 "" H 12638 6450 50  0001 C CNN
 F 3 "~" H 12600 6600 50  0001 C CNN
@@
 	12600 6800 12600 6750
 Wire Wire Line
-	14400 6400 13850 6400
+	14200 6400 13850 6400
 Wire Wire Line
 	11400 6400 12050 6400
-$Comp
-L 74xx:74HC7014 U?
-U 2 1 5C097319
-P 13550 5150
-F 0 "U?" H 13550 5467 50  0000 C CNN
-F 1 "74HC7014" H 13550 5376 50  0000 C CNN
-F 2 "Package_SO:SOIC-14_3.9x8.7mm_P1.27mm" H 13550 5150 50  0001 C CNN
-F 3 "https://assets.nexperia.com/documents/data-sheet/74HC7014.pdf" H 13550 5150 50  0001 C CNN
-	2    13550 5150
-	1    0    0    -1
-$EndComp
-$Comp
-L 74xx:74HC7014 U?
-U 3 1 5C097320
-P 13550 6400
-F 0 "U?" H 13550 6717 50  0000 C CNN
-F 1 "74HC7014" H 13550 6626 50  0000 C CNN
-F 2 "Package_SO:SOIC-14_3.9x8.7mm_P1.27mm" H 13550 6400 50  0001 C CNN
-F 3 "https://assets.nexperia.com/documents/data-sheet/74HC7014.pdf" H 13550 6400 50  0001 C CNN
-	3    13550 6400
-	1    0    0    -1
-$EndComp
 Text Label 12800 5150 0    50   ~ 0
 B_ABN_TVS
@@
 N_ABN_TVS
 Text HLabel 15650 6650 2    50   Output ~ 0
-A_ABN
+ENC_A
 Text HLabel 15650 6750 2    50   Output ~ 0
-B_ABN
+ENC_B
 Text HLabel 15650 6850 2    50   Output ~ 0
-N_ABN
-Wire Wire Line
-	15650 6650 15050 6650
-Wire Wire Line
-	15050 6750 15650 6750
-Wire Wire Line
-	15050 6850 15650 6850
+ENC_N
+Wire Wire Line
+	15650 6650 15350 6650
+Wire Wire Line
+	15350 6750 15650 6750
+Wire Wire Line
+	15350 6850 15650 6850
 Text Label 11400 3900 0    50   ~ 0
-A_ABN_i
+ENC_A_i
 Text Label 11400 5150 0    50   ~ 0
-B_ABN_i
+ENC_B_i
 Text Label 11400 6400 0    50   ~ 0
-N_ABN_i
+ENC_N_i
+Text Notes 9250 3450 0    50   ~ 0
+Lowpass filters set for about 72Khz\nSchmitt trigger inputs for taking out noise
+Text Notes 12900 3450 0    50   ~ 0
+Lowpass filters set for about 1.59Khz\nSchmitt trigger inputs for taking out noise
+$Comp
+L MotorControllerParts:R R?
+U 1 1 5D302326
+P 12200 6400
+F 0 "R?" V 12100 6350 50  0000 L CNN
+F 1 "100R" V 12300 6300 50  0000 L CNN
+F 2 "" V 12130 6400 50  0001 C CNN
+F 3 "~" H 12200 6400 50  0001 C CNN
+	1    12200 6400
+	0    1    1    0
+$EndComp
+$Comp
+L MotorControllerParts:R R?
+U 1 1 5D3026B7
+P 8600 6400
+F 0 "R?" V 8500 6350 50  0000 L CNN
+F 1 "100R" V 8700 6300 50  0000 L CNN
+F 2 "" V 8530 6400 50  0001 C CNN
+F 3 "~" H 8600 6400 50  0001 C CNN
+	1    8600 6400
+	0    1    1    0
+$EndComp
+$Comp
+L MotorControllerParts:R R?
+U 1 1 5D3027D9
+P 8600 5150
+F 0 "R?" V 8500 5100 50  0000 L CNN
+F 1 "100R" V 8700 5050 50  0000 L CNN
+F 2 "" V 8530 5150 50  0001 C CNN
+F 3 "~" H 8600 5150 50  0001 C CNN
+	1    8600 5150
+	0    1    1    0
+$EndComp
+$Comp
+L MotorControllerParts:R R?
+U 1 1 5D3028AB
+P 8600 3900
+F 0 "R?" V 8500 3850 50  0000 L CNN
+F 1 "100R" V 8700 3800 50  0000 L CNN
+F 2 "" V 8530 3900 50  0001 C CNN
+F 3 "~" H 8600 3900 50  0001 C CNN
+	1    8600 3900
+	0    1    1    0
+$EndComp
+Text Label 15350 6650 0    50   ~ 0
+ENC_A
+Text Label 15350 6750 0    50   ~ 0
+ENC_B
+Text Label 15350 6850 0    50   ~ 0
+ENC_N
+Text Label 14200 3900 2    50   ~ 0
+ENC_A
+Text Label 14200 5150 2    50   ~ 0
+ENC_B
+Text Label 14200 6400 2    50   ~ 0
+ENC_N
+Text Label 1750 7250 2    50   ~ 0
+ENC_N_i
+Text Label 1750 7150 2    50   ~ 0
+ENC_B_i
+Text Label 1750 7050 2    50   ~ 0
+ENC_A_i
 $EndSCHEMATC

Commit message: Working schematics
Parts:
- renumbered C501 to C401, C502 to C402, C503 to C403, C504 to C404, C505 to C405, C506 to C406, C507 to C407, C508 to C408, C509 to C409, C510 to C410, C511 to C411, C512 to C412, C513 to C413, C514 to C414, R501 to R401, R502 to R402, R503 to R403, R504 to R404, R505 to R405, R506 to R406, R508 to R408, R510 to R410, U501 to U401, U502 to U402, U503 to U403, U504 to U404, U506 to U406
Connections:
- net labels removed: A_ABN_TVS, A_HALL_TVS, B_ABN_TVS, B_HALL_TVS, N_ABN_TVS
Other:
- note added: "This sheet contains input/output proteciton and conditioning circuitry. \nNote that the stm32 USB lines pass through this sheet\nwithout modification."
- note removed: "Lowpass filters set for about 72Khz\nSchmitt trigger inputs for taking out noise"
- note removed: "This sheet contains input/output proteciton and conditioning circuitry. \nNote that the TMC4671 and stm32 USB lines pass through this sheet\nwithout modification."

Commit message: Compacted schematic layout
Parts:
- gave numbers to parts that had none: 19
- renumbered C401 to C201, C402 to C202, C403 to C203, C404 to C204, C405 to C205, C406 to C206, C407 to C207, C408 to C208, C409 to C209, C410 to C210, C411 to C211, C412 to C212, C413 to C213, C414 to C214, JP502 to JP201, R401 to R201, R402 to R202, R403 to R203, R404 to R204, R405 to R205, R406 to R206, R408 to R216, R410 to R220, U401 to U201, U402 to U202, U403 to U203, U404 to U204, U406 to U206

Commit message: Moved all parts into the MotorControllerParts.lib file
Parts:
- U204, U205: symbol 74xx:74HC7014 -> MotorControllerParts:74HC7014
Changed lines of the file:
@@
 Phase_A_HALL
 $Comp
-L 74xx:74HC7014 U205
+L MotorControllerParts:74HC7014 U205
 U 1 1 5CCC1B5B
 P 9950 3900
@@
 $EndComp
 $Comp
-L 74xx:74HC7014 U204
+L MotorControllerParts:74HC7014 U204
 U 1 1 5CCE6839
 P 8500 1250

Commit message: Added footprints, changed pdf
Parts:
- C201, C202, C203, C204, C205, C206, C207, C208, C209, C210, C211, C212, C213, C214, C215, C216, C217, C218, C219, C220: footprint (none) -> Capacitor_SMD:C_0805_2012Metric_Pad1.15x1.40mm_HandSolder
- JP201: footprint (none) -> Connector_PinHeader_2.54mm:PinHeader_1x02_P2.54mm_Vertical
- R201, R202, R203, R204, R205, R206, R207, R208, R209, R210, R211, R212, R213, R214, R215, R216, R217, R218, R219, R220: footprint (none) -> Resistor_SMD:R_0805_2012Metric_Pad1.15x1.40mm_HandSolder
- U201, U202, U203: footprint (none) -> Package_SO:SOIC-14_3.9x8.7mm_P1.27mm
- U206: footprint (none) -> Package_SO:SOIC-8_3.9x4.9mm_P1.27mm
