File: motor-controller-hw/IO.sch (KiCad schematic (older format))
At the start: 47 parts, among them U201 MCP6004, U202 MCP6004, U203 MCP6004, U204 74HC7014, U205 74HC7014, U206 mcp2562

Commit message: Adding BOM, changed some footprints -Changed footprints to linux models in schematics -Added field Digi-key# to all components -Started filling in said field
Parts:
- C201, C204, C205, C206, C207, C208, C209, C210, C211: footprint Capacitor_SMD:C_0805_2012Metric_Pad1.15x1.40mm_HandSolder -> Capacitors_SMD:C_0805_HandSoldering; Digi-key# (none) -> 1276-2444-1-ND
- C202, C212, C213: footprint Capacitor_SMD:C_0805_2012Metric_Pad1.15x1.40mm_HandSolder -> Capacitors_SMD:C_0805_HandSoldering; Digi-key# (none) -> 732-7672-1-ND
- C203: value 160n -> 150n; footprint Capacitor_SMD:C_0805_2012Metric_Pad1.15x1.40mm_HandSolder -> Capacitors_SMD:C_0805_HandSoldering; Digi-key# (none) -> 732-7674-1-ND
- C214: value 10u -> 4u7; footprint Capacitor_SMD:C_0805_2012Metric_Pad1.15x1.40mm_HandSolder -> Capacitors_SMD:C_0805_HandSoldering; Digi-key# (none) -> 732-7628-1-ND
- C215, C216, C217, C218, C219, C220: value 100n -> 100p; footprint Capacitor_SMD:C_0805_2012Metric_Pad1.15x1.40mm_HandSolder -> Capacitors_SMD:C_0805_HandSoldering; Digi-key# (none) -> 1276-1014-1-ND
- JP201: value CAN Termination -> CAN Term
- R201, R202, R203, R204, R205, R206, R207, R208, R209, R210, R211, R212, R213, R214, R215, R216, R217, R218, R219, R220: footprint Resistor_SMD:R_0805_2012Metric_Pad1.15x1.40mm_HandSolder -> Resistors_SMD:R_0805_HandSoldering
- U201, U202, U203: Digi-key# (none) -> MCP6004-I/SL-ND‎
- U204, U205: symbol 74xx:74HC7014 -> MotorControllerParts:74HC7014; Digi-key# (none) -> 1727-6342-1-ND
- U205: Digi-key# (none) -> 1727-6342-1-ND
- U206: Digi-key# (none) -> 568-11881-1-ND
Other:
- note added: "Schmitt trigger inputs for taking out noise"
- note removed: "Lowpass filters set for about 1.59Khz\nSchmitt trigger inputs for taking out noise"

Commit message: Moved some parts into the project parts library messed with the PCB slightly
Parts:
- U204, U205: symbol 74xx:74HC7014 -> MotorControllerParts:74HC7014
Changed lines of the file:
@@
 $EndComp
 $Comp
-L power:GNDD #PWR0227
+L MotorControllerParts:GNDD #PWR0227
 U 1 1 5D21A1B7
 P 13200 2500
+AR Path="/5D21A1B7" Ref="#PWR0227"  Part="1"
+AR Path="/5BB2528B/5D21A1B7" Ref="#PWR0227"  Part="1"
 F 0 "#PWR0227" H 13200 2250 50  0001 C CNN
 F 1 "GNDD" H 13204 2345 50  0000 C CNN
@@
 	13950 2000 13950 2100
 $Comp
-L power:GNDD #PWR0229
+L MotorControllerParts:GNDD #PWR0229
 U 1 1 5D3AC1DB
 P 13950 2500
+AR Path="/5D3AC1DB" Ref="#PWR0229"  Part="1"
+AR Path="/5BB2528B/5D3AC1DB" Ref="#PWR0229"  Part="1"
 F 0 "#PWR0229" H 13950 2250 50  0001 C CNN
 F 1 "GNDD" H 13954 2345 50  0000 C CNN
@@
 $EndComp
 $Comp
-L 74xx:74HC7014 U205
+L MotorControllerParts:74HC7014 U205
 U 7 1 5CCC2847
 P 5250 8950
+AR Path="/5CCC2847" Ref="U205"  Part="7"
+AR Path="/5BB2528B/5CCC2847" Ref="U205"  Part="7"
 F 0 "U205" H 5150 9000 50  0000 L CNN
 F 1 "74HC7014" V 5000 8750 50  0000 L CNN
@@
 $EndComp
 $Comp
-L 74xx:74HC7014 U204
+L MotorControllerParts:74HC7014 U204
 U 2 1 5CCE6840
 P 10100 1250
+AR Path="/5CCE6840" Ref="U204"  Part="2"
+AR Path="/5BB2528B/5CCE6840" Ref="U204"  Part="2"
 F 0 "U204" H 10100 1567 50  0000 C CNN
 F 1 "74HC7014" H 10100 1476 50  0000 C CNN

Commit message: Added all of the digi-key part numbers
Parts:
- JP201: Digi-key# (none) -> S1212EC-02-ND
- R201, R202, R203, R204, R205: Digi-key# (none) -> A126358CT-ND
- R206: Digi-key# (none) -> 311-3.90CRCT-ND
- R207, R208, R209, R213, R214, R215: Digi-key# (none) -> 311-100CRCT-ND
- R210, R211, R212, R217, R218, R219: Digi-key# (none) -> 311-4.70KCRCT-ND
- R216: Digi-key# (none) -> A129738CT-ND
- R220: Digi-key# (none) -> A129761CT-ND
Changed lines of the file:
@@
 F 1 "2K" V 4650 1500 50  0000 C CNN
 F 2 "Resistors_SMD:R_0805_HandSoldering" V 4580 1500 50  0001 C CNN
-F 3 "~" H 4650 1500 50  0001 C CNN
+F 3 "https://www.te.com/commerce/DocumentDelivery/DDEController?Action=srchrtrv&DocNm=1773204&DocType=DS&DocLang=English" H 4650 1500 50  0001 C CNN
+F 4 "A126358CT-ND" H 0   0   50  0001 C CNN "Digi-key#"
 	1    4650 1500
 	0    1    1    0
@@
 F 1 "3K9" V 4850 1750 50  0000 C CNN
 F 2 "Resistors_SMD:R_0805_HandSoldering" V 4780 1750 50  0001 C CNN
-F 3 "~" H 4850 1750 50  0001 C CNN
+F 3 "http://www.yageo.com/documents/recent/PYu-RC_Group_51_RoHS_L_9.pdf" H 4850 1750 50  0001 C CNN
+F 4 "311-3.90CRCT-ND" H 0   0   50  0001 C CNN "Digi-key#"
 	1    4850 1750
 	-1   0    0    1
@@
 F 1 "2K" V 4650 2500 50  0000 C CNN
 F 2 "Resistors_SMD:R_0805_HandSoldering" V 4580 2500 50  0001 C CNN
-F 3 "~" H 4650 2500 50  0001 C CNN
+F 3 "https://www.te.com/commerce/DocumentDelivery/DDEController?Action=srchrtrv&DocNm=1773204&DocType=DS&DocLang=English" H 4650 2500 50  0001 C CNN
+F 4 "A126358CT-ND" H 0   0   50  0001 C CNN "Digi-key#"
 	1    4650 2500
 	0    1    1    0
@@
 F 1 "2K" V 4650 3450 50  0000 C CNN
 F 2 "Resistors_SMD:R_0805_HandSoldering" V 4580 3450 50  0001 C CNN
-F 3 "~" H 4650 3450 50  0001 C CNN
+F 3 "https://www.te.com/commerce/DocumentDelivery/DDEController?Action=srchrtrv&DocNm=1773204&DocType=DS&DocLang=English" H 4650 3450 50  0001 C CNN
+F 4 "A126358CT-ND" H 0   0   50  0001 C CNN "Digi-key#"
 	1    4650 3450
 	0    1    1    0
@@
 F 1 "2K" V 4650 4400 50  0000 C CNN
 F 2 "Resistors_SMD:R_0805_HandSoldering" V 4580 4400 50  0001 C CNN
-F 3 "~" H 4650 4400 50  0001 C CNN
+F 3 "https://www.te.com/commerce/DocumentDelivery/DDEController?Action=srchrtrv&DocNm=1773204&DocType=DS&DocLang=English" H 4650 4400 50  0001 C CNN
+F 4 "A126358CT-ND" H 0   0   50  0001 C CNN "Digi-key#"
 	1    4650 4400
 	0    1    1    0
@@
 F 1 "2K" V 4650 5350 50  0000 C CNN
 F 2 "Resistors_SMD:R_0805_HandSoldering" V 4580 5350 50  0001 C CNN
-F 3 "~" H 4650 5350 50  0001 C CNN
+F 3 "https://www.te.com/commerce/DocumentDelivery/DDEController?Action=srchrtrv&DocNm=1773204&DocType=DS&DocLang=English" H 4650 5350 50  0001 C CNN
+F 4 "A126358CT-ND" H 0   0   50  0001 C CNN "Digi-key#"
 	1    4650 5350
 	0    1    1    0
@@
 F 1 "120R" V 12400 2350 50  0000 C CNN
 F 2 "Resistors_SMD:R_0805_HandSoldering" V 12230 2350 50  0001 C CNN
-F 3 "~" H 12300 2350 50  0001 C CNN
+F 3 "https://www.te.com/commerce/DocumentDelivery/DDEController?Action=srchrtrv&DocNm=1773204-3&DocType=DS&DocLang=English" H 12300 2350 50  0001 C CNN
+F 4 "A129738CT-ND" H 0   0   50  0001 C CNN "Digi-key#"
 	1    12300 2350
 	0    1    1    0
@@
 F 1 "CAN Term" H 12000 2250 50  0000 C CNN
 F 2 "Connector_PinHeader_2.54mm:PinHeader_1x02_P2.54mm_Vertical" H 12000 2350 50  0001 C CNN
-F 3 "~" H 12000 2350 50  0001 C CNN
+F 3 "https://media.digikey.com/PDF/Data%20Sheets/Sullins%20PDFs/xRxCzzzSxxN-RC_ST_11635-B.pdf" H 12000 2350 50  0001 C CNN
+F 4 "S1212EC-02-ND" H 0   0   50  0001 C CNN "Digi-key#"
 	1    12000 2350
 	1    0    0    -1
@@
 F 1 "10K" H 13880 2295 50  0000 R CNN
 F 2 "Resistors_SMD:R_0805_HandSoldering" V 13880 2250 50  0001 C CNN
-F 3 "~" H 13950 2250 50  0001 C CNN
+F 3 "https://www.te.com/commerce/DocumentDelivery/DDEController?Action=srchrtrv&DocNm=1773204-3&DocType=DS&DocLang=English" H 13950 2250 50  0001 C CNN
+F 4 "A129761CT-ND" H 0   0   50  0001 C CNN "Digi-key#"
 	1    13950 2250
 	-1   0    0    1
@@
 F 1 "4K7" H 9050 3650 50  0000 L CNN
 F 2 "Resistors_SMD:R_0805_HandSoldering" V 8930 3700 50  0001 C CNN
-F 3 "~" H 9000 3700 50  0001 C CNN
+F 3 "http://www.yageo.com/documents/recent/PYu-RC_Group_51_RoHS_L_9.pdf" H 9000 3700 50  0001 C CNN
+F 4 "311-4.70KCRCT-ND" H 0   0   50  0001 C CNN "Digi-key#"
 	1    9000 3700
 	1    0    0    -1
@@
 F 1 "4K7" H 9050 4900 50  0000 L CNN
 F 2 "Resistors_SMD:R_0805_HandSoldering" V 8930 4950 50  0001 C CNN
-F 3 "~" H 9000 4950 50  0001 C CNN
+F 3 "http://www.yageo.com/documents/recent/PYu-RC_Group_51_RoHS_L_9.pdf" H 9000 4950 50  0001 C CNN
+F 4 "311-4.70KCRCT-ND" H 0   0   50  0001 C CNN "Digi-key#"
 	1    9000 4950
 	1    0    0    -1
@@
 F 1 "4K7" H 9050 6150 50  0000 L CNN
 F 2 "Resistors_SMD:R_0805_HandSoldering" V 8930 6200 50  0001 C CNN
-F 3 "~" H 9000 6200 50  0001 C CNN
+F 3 "http://www.yageo.com/documents/recent/PYu-RC_Group_51_RoHS_L_9.pdf" H 9000 6200 50  0001 C CNN
+F 4 "311-4.70KCRCT-ND" H 0   0   50  0001 C CNN "Digi-key#"
 	1    9000 6200
 	1    0    0    -1
@@
 F 1 "100R" V 12300 3800 50  0000 L CNN
 F 2 "Resistors_SMD:R_0805_HandSoldering" V 12130 3900 50  0001 C CNN
-F 3 "~" H 12200 3900 50  0001 C CNN
+F 3 "http://www.yageo.com/documents/recent/PYu-RC_Group_51_RoHS_L_9.pdf" H 12200 3900 50  0001 C CNN
+F 4 "311-100CRCT-ND" H 0   0   50  0001 C CNN "Digi-key#"
 	1    12200 3900
 	0    1    1    0
@@
 F 1 "4K7" H 12650 3650 50  0000 L CNN
 F 2 "Resistors_SMD:R_0805_HandSoldering" V 12530 3700 50  0001 C CNN
-F 3 "~" H 12600 3700 50  0001 C CNN
+F 3 "http://www.yageo.com/documents/recent/PYu-RC_Group_51_RoHS_L_9.pdf" H 12600 3700 50  0001 C CNN
+F 4 "311-4.70KCRCT-ND" H 0   0   50  0001 C CNN "Digi-key#"
 	1    12600 3700
 	1    0    0    -1
@@
 F 1 "100R" V 12300 5050 50  0000 L CNN
 F 2 "Resistors_SMD:R_0805_HandSoldering" V 12130 5150 50  0001 C CNN
-F 3 "~" H 12200 5150 50  0001 C CNN
+F 3 "http://www.yageo.com/documents/recent/PYu-RC_Group_51_RoHS_L_9.pdf" H 12200 5150 50  0001 C CNN
+F 4 "311-100CRCT-ND" H 0   0   50  0001 C CNN "Digi-key#"
 	1    12200 5150
 	0    1    1    0
@@
 F 1 "4K7" H 12650 4900 50  0000 L CNN
 F 2 "Resistors_SMD:R_0805_HandSoldering" V 12530 4950 50  0001 C CNN
-F 3 "~" H 12600 4950 50  0001 C CNN
+F 3 "http://www.yageo.com/documents/recent/PYu-RC_Group_51_RoHS_L_9.pdf" H 12600 4950 50  0001 C CNN
+F 4 "311-4.70KCRCT-ND" H 0   0   50  0001 C CNN "Digi-key#"
 	1    12600 4950
 	1    0    0    -1
@@
 F 1 "4K7" H 12650 6150 50  0000 L CNN
 F 2 "Resistors_SMD:R_0805_HandSoldering" V 12530 6200 50  0001 C CNN
-F 3 "~" H 12600 6200 50  0001 C CNN
+F 3 "http://www.yageo.com/documents/recent/PYu-RC_Group_51_RoHS_L_9.pdf" H 12600 6200 50  0001 C CNN
+F 4 "311-4.70KCRCT-ND" H 0   0   50  0001 C CNN "Digi-key#"
 	1    12600 6200
 	1    0    0    -1
@@
 F 1 "100R" V 12300 6300 50  0000 L CNN
 F 2 "Resistors_SMD:R_0805_HandSoldering" V 12130 6400 50  0001 C CNN
-F 3 "~" H 12200 6400 50  0001 C CNN
+F 3 "http://www.yageo.com/documents/recent/PYu-RC_Group_51_RoHS_L_9.pdf" H 12200 6400 50  0001 C CNN
+F 4 "311-100CRCT-ND" H 0   0   50  0001 C CNN "Digi-key#"
 	1    12200 6400
 	0    1    1    0
@@
 F 1 "100R" V 8700 6300 50  0000 L CNN
 F 2 "Resistors_SMD:R_0805_HandSoldering" V 8530 6400 50  0001 C CNN
-F 3 "~" H 8600 6400 50  0001 C CNN
+F 3 "http://www.yageo.com/documents/recent/PYu-RC_Group_51_RoHS_L_9.pdf" H 8600 6400 50  0001 C CNN
+F 4 "311-100CRCT-ND" H 0   0   50  0001 C CNN "Digi-key#"
 	1    8600 6400
 	0    1    1    0
@@
 F 1 "100R" V 8700 5050 50  0000 L CNN
 F 2 "Resistors_SMD:R_0805_HandSoldering" V 8530 5150 50  0001 C CNN
-F 3 "~" H 8600 5150 50  0001 C CNN
+F 3 "http://www.yageo.com/documents/recent/PYu-RC_Group_51_RoHS_L_9.pdf" H 8600 5150 50  0001 C CNN
+F 4 "311-100CRCT-ND" H 0   0   50  0001 C CNN "Digi-key#"
 	1    8600 5150
 	0    1    1    0
@@
 F 1 "100R" V 8700 3800 50  0000 L CNN
 F 2 "Resistors_SMD:R_0805_HandSoldering" V 8530 3900 50  0001 C CNN
-F 3 "~" H 8600 3900 50  0001 C CNN
+F 3 "http://www.yageo.com/documents/recent/PYu-RC_Group_51_RoHS_L_9.pdf" H 8600 3900 50  0001 C CNN
+F 4 "311-100CRCT-ND" H 0   0   50  0001 C CNN "Digi-key#"
 	1    8600 3900
 	0    1    1    0
