File: motor-controller-hw/motor-controller-hw.kicad_pcb (KiCad board)
At the start: 4 copper layers, 99.7 x 85.1 mm, 175 parts, among them J101 CAN, J102 Throttle, J103 Motor T, J104 Tran T, J105 USB_B_Micro, J106 Extra IO, J107 Hall Sensors, J108 CAN_DBG, J109 ABN Encoder, J110 SPI_DBG, J111 Trinamic-Bridge, J301 SWD, J302 User USART, J401 Trinamic_TRMI, J402 TMC4671 USART, Q101 Q_PMOS_GDS, SW301 Reset, SW302 Boot, SW303 User_SW, U101 AP7361C-33, U102 D36V6F5, U201 MCP6004, U202 MCP6004, U203 MCP6004, U204 74HC7014, U205 74HC7014, U206 mcp2562, U301 STM32F303RETx, U401 TMC4671, X401 IQXO-50, Y301 8Mhz

Commit message: Fixed pad clearance issues
Parts:
- C105, C214: value 10u -> 4u7
- C203: value 160n -> 150n
- C309, C310: value 26pf -> 27pf
- D101: value 18V Zener -> 15V Zener
- R105, R306, R307: value 510R -> 330R
- R302: value 390R -> 330R
- R305: value 510R -> 100R
Other:
- rule pad_to_mask_clearance: 0.2 -> 0.0381
- rule solder_mask_min_width: 0.25 -> 0.00254
Changed lines of the file:
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@@
     (pad_size 6.4 6.4)
     (pad_drill 3.2)
-    (pad_to_mask_clearance 0.2)
-    (solder_mask_min_width 0.25)
+    (pad_to_mask_clearance 0.0381)
+    (solder_mask_min_width 0.00254)
     (aux_axis_origin 0 0)
     (visible_elements 7FFFFF7F)
@@
       (effects (font (size 1 1) (thickness 0.15)) (justify mirror))
     )
-    (fp_text value 10u (at 0 -1.65 180) (layer B.Fab)
+    (fp_text value 4u7 (at 0 -1.65 180) (layer B.Fab)
       (effects (font (size 1 1) (thickness 0.15)) (justify mirror))
     )
@@
       (effects (font (size 1 1) (thickness 0.15)) (justify mirror))
     )
-    (fp_text value 160n (at 0 -1.65) (layer B.Fab)
+    (fp_text value 150n (at 0 -1.65) (layer B.Fab)
       (effects (font (size 1 1) (thickness 0.15)) (justify mirror))
     )
@@
       (effects (font (size 1 1) (thickness 0.15)) (justify mirror))
     )
-    (fp_text value 10u (at 0 2.54 90) (layer B.Fab)
+    (fp_text value 4u7 (at 0 2.54 90) (layer B.Fab)
       (effects (font (size 1 1) (thickness 0.15)) (justify mirror))
     )
@@
       (effects (font (size 1 1) (thickness 0.15)) (justify mirror))
     )
-    (fp_text value 26pf (at 0 -1.65 270) (layer B.Fab)
+    (fp_text value 27pf (at 0 -1.65 270) (layer B.Fab)
       (effects (font (size 1 1) (thickness 0.15)) (justify mirror))
     )
@@
       (effects (font (size 1 1) (thickness 0.15)) (justify mirror))
     )
-    (fp_text value 26pf (at 0 -1.65 90) (layer B.Fab)
+    (fp_text value 27pf (at 0 -1.65 90) (layer B.Fab)
       (effects (font (size 1 1) (thickness 0.15)) (justify mirror))
     )
@@
       (effects (font (size 1 1) (thickness 0.15)) (justify mirror))
     )
-    (fp_text value "18V Zener" (at 0 -2.1) (layer B.Fab)
+    (fp_text value "15V Zener" (at 0 -2.1) (layer B.Fab)
       (effects (font (size 1 1) (thickness 0.15)) (justify mirror))
     )
@@
       (effects (font (size 1 1) (thickness 0.15)))
     )
-    (fp_text value 390R (at 0 1.65 270) (layer F.Fab)
+    (fp_text value 330R (at 0 1.65 270) (layer F.Fab)
       (effects (font (size 1 1) (thickness 0.15)))
     )
@@
       (effects (font (size 1 1) (thickness 0.15)))
     )
-    (fp_text value 510R (at 0 1.65 90) (layer F.Fab)
+    (fp_text value 100R (at 0 1.65 90) (layer F.Fab)
       (effects (font (size 1 1) (thickness 0.15)))
     )
@@
       (effects (font (size 1 1) (thickness 0.15)))
     )
-    (fp_text value 510R (at 0 1.65 90) (layer F.Fab)
+    (fp_text value 330R (at 0 1.65 90) (layer F.Fab)
       (effects (font (size 1 1) (thickness 0.15)))
     )
@@
       (effects (font (size 1 1) (thickness 0.15)))
     )
-    (fp_text value 510R (at 0 1.65 90) (layer F.Fab)
+    (fp_text value 330R (at 0 1.65 90) (layer F.Fab)
       (effects (font (size 1 1) (thickness 0.15)))
     )
@@
   (module supermileage_footprints:TMC4671 (layer F.Cu)
     (at 106.426 88.9762)
+    (solder_mask_margin 0.0381)
+    (solder_paste_margin -0.00254)
     (clearance 0.075)
     (attr smd)
@@
       (effects (font (size 1 1) (thickness 0.15)))
     )
-    (fp_text value 510R (at 0 1.75 90) (layer F.Fab)
+    (fp_text value 330R (at 0 1.75 90) (layer F.Fab)
       (effects (font (size 1 1) (thickness 0.15)))
     )
