File: motor-controller-hw/microcontroller.sch (KiCad schematic (older format))
At the start: 28 parts, among them J301 SWD, J302 User USART, SW301 Reset, SW302 Boot, SW303 User_SW, U301 STM32F303RETx, Y301 8Mhz

Commit message: Adding BOM, changed some footprints -Changed footprints to linux models in schematics -Added field Digi-key# to all components -Started filling in said field
Parts:
- C301, C302, C303, C304, C305, C311: footprint Capacitor_SMD:C_0805_2012Metric_Pad1.15x1.40mm_HandSolder -> Capacitors_SMD:C_0805_HandSoldering; Digi-key# (none) -> 1276-2444-1-ND
- C306: footprint Capacitor_SMD:C_0805_2012Metric_Pad1.15x1.40mm_HandSolder -> Capacitors_SMD:C_0805_HandSoldering; Digi-key# (none) -> 732-7628-1-ND
- C307: footprint Capacitor_SMD:C_0805_2012Metric_Pad1.15x1.40mm_HandSolder -> Capacitors_SMD:C_0805_HandSoldering; Digi-key# (none) -> 732-7672-1-ND
- C308: footprint Capacitor_SMD:C_0805_2012Metric_Pad1.15x1.40mm_HandSolder -> Capacitors_SMD:C_0805_HandSoldering; Digi-key# (none) -> 732-12169-1-ND
- C309, C310: value 26pf -> 27pf; footprint Capacitor_SMD:C_0805_2012Metric_Pad1.15x1.40mm_HandSolder -> Capacitors_SMD:C_0805_HandSoldering; Digi-key# (none) -> 1276-2622-1-ND
- R301, R302, R303, R304, R305, R306, R307: footprint Resistor_SMD:R_0805_2012Metric_Pad1.15x1.40mm_HandSolder -> Resistors_SMD:R_0805_HandSoldering
- SW301, SW302, SW303: Digi-key# (none) -> 450-1758-1-ND
- U301: Digi-key# (none) -> 497-15163-ND
- Y301: Digi-key# (none) -> 535-10212-1-ND‎
Connections:
- no-connect marks 12 -> 13
Changed lines of the file:
@@
 F 2 "Package_QFP:LQFP-64_10x10mm_P0.5mm" H 4800 1200 50  0001 R CNN
 F 3 "http://www.st.com/st-web-ui/static/active/en/resource/technical/document/datasheet/DM00118585.pdf" H 5400 2900 50  0001 C CNN
+F 4 "497-15163-ND" H 5400 2900 50  0001 C CNN "Digi-key#"
 	1    5400 2900
 	1    0    0    -1
@@
 F 0 "C301" H 950 7350 50  0000 L CNN
 F 1 "100n" H 950 7150 50  0000 L CNN
-F 2 "Capacitor_SMD:C_0805_2012Metric_Pad1.15x1.40mm_HandSolder" H 938 7100 50  0001 C CNN
+F 2 "Capacitors_SMD:C_0805_HandSoldering" H 938 7100 50  0001 C CNN
 F 3 "~" H 900 7250 50  0001 C CNN
+F 4 "1276-2444-1-ND" H 900 7250 50  0001 C CNN "Digi-key#"
 	1    900  7250
 	1    0    0    -1
@@
 F 0 "C302" H 1300 7350 50  0000 L CNN
 F 1 "100n" H 1300 7150 50  0000 L CNN
-F 2 "Capacitor_SMD:C_0805_2012Metric_Pad1.15x1.40mm_HandSolder" H 1288 7100 50  0001 C CNN
+F 2 "Capacitors_SMD:C_0805_HandSoldering" H 1288 7100 50  0001 C CNN
 F 3 "~" H 1250 7250 50  0001 C CNN
+F 4 "1276-2444-1-ND" H 1250 7250 50  0001 C CNN "Digi-key#"
 	1    1250 7250
 	1    0    0    -1
@@
 F 0 "C304" H 1650 7350 50  0000 L CNN
 F 1 "100n" H 1650 7150 50  0000 L CNN
-F 2 "Capacitor_SMD:C_0805_2012Metric_Pad1.15x1.40mm_HandSolder" H 1638 7100 50  0001 C CNN
+F 2 "Capacitors_SMD:C_0805_HandSoldering" H 1638 7100 50  0001 C CNN
 F 3 "~" H 1600 7250 50  0001 C CNN
+F 4 "1276-2444-1-ND" H 1600 7250 50  0001 C CNN "Digi-key#"
 	1    1600 7250
 	1    0    0    -1
@@
 F 0 "C305" H 2000 7350 50  0000 L CNN
 F 1 "100n" H 2000 7150 50  0000 L CNN
-F 2 "Capacitor_SMD:C_0805_2012Metric_Pad1.15x1.40mm_HandSolder" H 1988 7100 50  0001 C CNN
+F 2 "Capacitors_SMD:C_0805_HandSoldering" H 1988 7100 50  0001 C CNN
 F 3 "~" H 1950 7250 50  0001 C CNN
+F 4 "1276-2444-1-ND" H 1950 7250 50  0001 C CNN "Digi-key#"
 	1    1950 7250
 	1    0    0    -1
@@
 F 0 "C306" H 2350 7350 50  0000 L CNN
 F 1 "4u7" H 2350 7150 50  0000 L CNN
-F 2 "Capacitor_SMD:C_0805_2012Metric_Pad1.15x1.40mm_HandSolder" H 2338 7100 50  0001 C CNN
+F 2 "Capacitors_SMD:C_0805_HandSoldering" H 2338 7100 50  0001 C CNN
 F 3 "~" H 2300 7250 50  0001 C CNN
+F 4 "732-7628-1-ND" H 2300 7250 50  0001 C CNN "Digi-key#"
 	1    2300 7250
 	1    0    0    -1
@@
 F 0 "C308" H 3250 7350 50  0000 L CNN
 F 1 "10n" H 3250 7150 50  0000 L CNN
-F 2 "Capacitor_SMD:C_0805_2012Metric_Pad1.15x1.40mm_HandSolder" H 3238 7100 50  0001 C CNN
+F 2 "Capacitors_SMD:C_0805_HandSoldering" H 3238 7100 50  0001 C CNN
 F 3 "~" H 3200 7250 50  0001 C CNN
+F 4 "732-12169-1-ND" H 3200 7250 50  0001 C CNN "Digi-key#"
 	1    3200 7250
 	1    0    0    -1
@@
 F 0 "C307" H 2950 7350 50  0000 L CNN
 F 1 "1u" H 2950 7150 50  0000 L CNN
-F 2 "Capacitor_SMD:C_0805_2012Metric_Pad1.15x1.40mm_HandSolder" H 2938 7100 50  0001 C CNN
+F 2 "Capacitors_SMD:C_0805_HandSoldering" H 2938 7100 50  0001 C CNN
 F 3 "~" H 2900 7250 50  0001 C CNN
+F 4 "732-7672-1-ND" H 2900 7250 50  0001 C CNN "Digi-key#"
 	1    2900 7250
 	1    0    0    -1
@@
 F 1 "8Mhz" V 7600 5850 50  0000 C CNN
 F 2 "Crystal:Crystal_SMD_HC49-SD_HandSoldering" H 7450 6000 50  0001 C CNN
-F 3 "~" H 7450 6000 50  0001 C CNN
+F 3 "https://abracon.com/Resonators/abls.pdf" H 7450 6000 50  0001 C CNN
+F 4 "535-10212-1-ND‎" H 7450 6000 50  0001 C CNN "Digi-key#"
 	1    7450 6000
 	0    -1   -1   0
@@
 P 7250 5750
 F 0 "C309" V 7200 5550 50  0000 L CNN
-F 1 "26pf" V 7350 5650 50  0000 L CNN
-F 2 "Capacitor_SMD:C_0805_2012Metric_Pad1.15x1.40mm_HandSolder" H 7250 5750 50  0001 C CNN
+F 1 "27pf" V 7350 5650 50  0000 L CNN
+F 2 "Capacitors_SMD:C_0805_HandSoldering" H 7250 5750 50  0001 C CNN
 F 3 "~" H 7250 5750 50  0001 C CNN
+F 4 "1276-2622-1-ND" H 7250 5750 50  0001 C CNN "Digi-key#"
 	1    7250 5750
 	0    1    1    0
@@
 P 7250 6250
 F 0 "C310" V 7200 6050 50  0000 L CNN
-F 1 "26pf" V 7350 6150 50  0000 L CNN
-F 2 "Capacitor_SMD:C_0805_2012Metric_Pad1.15x1.40mm_HandSolder" H 7250 6250 50  0001 C CNN
+F 1 "27pf" V 7350 6150 50  0000 L CNN
+F 2 "Capacitors_SMD:C_0805_HandSoldering" H 7250 6250 50  0001 C CNN
 F 3 "~" H 7250 6250 50  0001 C CNN
+F 4 "1276-2622-1-ND" H 7250 6250 50  0001 C CNN "Digi-key#"
 	1    7250 6250
 	0    1    1    0
@@
 F 0 "R302" V 7650 6250 50  0000 C CNN
 F 1 "390R" V 7850 6250 50  0000 C CNN
-F 2 "Resistor_SMD:R_0805_2012Metric_Pad1.15x1.40mm_HandSolder" H 7750 6250 50  0001 C CNN
+F 2 "Resistors_SMD:R_0805_HandSoldering" H 7750 6250 50  0001 C CNN
 F 3 "~" H 7750 6250 50  0001 C CNN
 	1    7750 6250
@@
 F 1 "Reset" V 1050 5750 50  0000 R CNN
 F 2 "supermileage_footprints:SW_SPST_FSMSM" H 900 5550 50  0001 C CNN
-F 3 "" H 900 5550 50  0001 C CNN
+F 3 "https://www.te.com/commerce/DocumentDelivery/DDEController?Action=srchrtrv&DocNm=1437566-3&DocType=Customer+Drawing&DocLang=English" H 900 5550 50  0001 C CNN
+F 4 "450-1758-1-ND" H 900 5550 50  0001 C CNN "Digi-key#"
 	1    900  5550
 	0    -1   -1   0
@@
 F 1 "Boot" V 2250 5450 50  0000 R CNN
 F 2 "supermileage_footprints:SW_SPST_FSMSM" H 2100 5250 50  0001 C CNN
-F 3 "" H 2100 5250 50  0001 C CNN
+F 3 "https://www.te.com/commerce/DocumentDelivery/DDEController?Action=srchrtrv&DocNm=1437566-3&DocType=Customer+Drawing&DocLang=English" H 2100 5250 50  0001 C CNN
+F 4 "450-1758-1-ND" H 2100 5250 50  0001 C CNN "Digi-key#"
 	1    2100 5250
 	0    -1   -1   0
@@
 F 0 "C303" H 1350 5700 50  0000 L CNN
 F 1 "100n" H 1350 5500 50  0000 L CNN
-F 2 "Capacitor_SMD:C_0805_2012Metric_Pad1.15x1.40mm_HandSolder" H 1338 5450 50  0001 C CNN
+F 2 "Capacitors_SMD:C_0805_HandSoldering" H 1338 5450 50  0001 C CNN
 F 3 "~" H 1300 5600 50  0001 C CNN
+F 4 "1276-2444-1-ND" H 1300 5600 50  0001 C CNN "Digi-key#"
 	1    1300 5600
 	1    0    0    -1
@@
 F 0 "R301" H 2070 5696 50  0000 L CNN
 F 1 "10K" H 2070 5605 50  0000 L CNN
-F 2 "Resistor_SMD:R_0805_2012Metric_Pad1.15x1.40mm_HandSolder" V 1930 5650 50  0001 C CNN
+F 2 "Resistors_SMD:R_0805_HandSoldering" V 1930 5650 50  0001 C CNN
 F 3 "~" H 2000 5650 50  0001 C CNN
 	1    2000 5650
@@
 F 0 "R307" V 9650 6300 50  0000 C CNN
 F 1 "510R" V 9434 6300 50  0000 C CNN
-F 2 "Resistor_SMD:R_0805_2012Metric_Pad1.15x1.40mm_HandSolder" V 9480 6300 50  0001 C CNN
+F 2 "Resistors_SMD:R_0805_HandSoldering" V 9480 6300 50  0001 C CNN
 F 3 "~" H 9550 6300 50  0001 C CNN
 	1    9550 6300
@@
 F 0 "R306" V 9650 5900 50  0000 C CNN
 F 1 "510R" V 9434 5900 50  0000 C CNN
-F 2 "Resistor_SMD:R_0805_2012Metric_Pad1.15x1.40mm_HandSolder" V 9480 5900 50  0001 C CNN
+F 2 "Resistors_SMD:R_0805_HandSoldering" V 9480 5900 50  0001 C CNN
 F 3 "~" H 9550 5900 50  0001 C CNN
 	1    9550 5900
@@
 F 0 "R305" V 9650 5500 50  0000 C CNN
 F 1 "510R" V 9434 5500 50  0000 C CNN
-F 2 "Resistor_SMD:R_0805_2012Metric_Pad1.15x1.40mm_HandSolder" V 9480 5500 50  0001 C CNN
+F 2 "Resistors_SMD:R_0805_HandSoldering" V 9480 5500 50  0001 C CNN
 F 3 "~" H 9550 5500 50  0001 C CNN
 	1    9550 5500
@@
 F 1 "User_SW" V 10350 4550 50  0000 R CNN
 F 2 "supermileage_footprints:SW_SPST_FSMSM" H 10100 4350 50  0001 C CNN
-F 3 "" H 10100 4350 50  0001 C CNN
+F 3 "https://www.te.com/commerce/DocumentDelivery/DDEController?Action=srchrtrv&DocNm=1437566-3&DocType=Customer+Drawing&DocLang=English" H 10100 4350 50  0001 C CNN
+F 4 "450-1758-1-ND" H 10100 4350 50  0001 C CNN "Digi-key#"
 	1    10100 4350
 	0    1    -1   0
@@
 F 0 "C311" H 9765 4496 50  0000 L CNN
 F 1 "100n" H 9765 4405 50  0000 L CNN
-F 2 "Capacitor_SMD:C_0805_2012Metric_Pad1.15x1.40mm_HandSolder" H 9688 4300 50  0001 C CNN
+F 2 "Capacitors_SMD:C_0805_HandSoldering" H 9688 4300 50  0001 C CNN
 F 3 "~" H 9650 4450 50  0001 C CNN
+F 4 "1276-2444-1-ND" H 9650 4450 50  0001 C CNN "Digi-key#"
 	1    9650 4450
 	1    0    0    -1
@@
 F 0 "R303" H 9720 4096 50  0000 L CNN
 F 1 "4K7" H 9720 4005 50  0000 L CNN
-F 2 "Resistor_SMD:R_0805_2012Metric_Pad1.15x1.40mm_HandSolder" V 9580 4050 50  0001 C CNN
+F 2 "Resistors_SMD:R_0805_HandSoldering" V 9580 4050 50  0001 C CNN
 F 3 "~" H 9650 4050 50  0001 C CNN
 	1    9650 4050
@@
 F 0 "R304" H 9720 4846 50  0000 L CNN
 F 1 "100R" H 9720 4755 50  0000 L CNN
-F 2 "Resistor_SMD:R_0805_2012Metric_Pad1.15x1.40mm_HandSolder" V 9580 4800 50  0001 C CNN
+F 2 "Resistors_SMD:R_0805_HandSoldering" V 9580 4800 50  0001 C CNN
 F 3 "~" H 9650 4800 50  0001 C CNN
 	1    9650 4800
@@
 NoConn ~ 4700 2800
 NoConn ~ 4700 4400
+NoConn ~ 6100 2300
 $EndSCHEMATC

Commit message: Added all of the digi-key part numbers
Parts:
- D301: Digi-key# (none) -> 732-12013-1-ND
- D302: Digi-key# (none) -> 732-12015-1-ND
- D303: Digi-key# (none) -> 732-12017-1-ND
- J301: Digi-key# (none) -> S1212EC-06-ND
- J302: Digi-key# (none) -> S1212EC-03-ND
- R301: Digi-key# (none) -> A129761CT-ND
- R302: value 390R -> 330R; symbol MotorControllerParts:R_Small -> MotorControllerParts:R; Digi-key# (none) -> 311-330CRCT-ND
- R303: Digi-key# (none) -> 311-4.70KCRCT-ND
- R304: Digi-key# (none) -> 311-100CRCT-ND
- R305: value 510R -> 100R; Digi-key# (none) -> 311-100CRCT-ND
- R306, R307: value 510R -> 330R; Digi-key# (none) -> 311-330CRCT-ND
Changed lines of the file:
@@
 U 1 1 5BF6BC78
 P 7450 6000
-F 0 "Y301" V 7450 5800 50  0000 C CNN
+F 0 "Y301" V 7450 5750 50  0000 C CNN
 F 1 "8Mhz" V 7600 5850 50  0000 C CNN
 F 2 "Crystal:Crystal_SMD_HC49-SD_HandSoldering" H 7450 6000 50  0001 C CNN
@@
 U 1 1 5BF6BDAE
 P 7250 5750
-F 0 "C309" V 7200 5550 50  0000 L CNN
+F 0 "C309" V 7150 5550 50  0000 L CNN
 F 1 "27pf" V 7350 5650 50  0000 L CNN
 F 2 "Capacitors_SMD:C_0805_HandSoldering" H 7250 5750 50  0001 C CNN
@@
 U 1 1 5BF6BDEC
 P 7250 6250
-F 0 "C310" V 7200 6050 50  0000 L CNN
+F 0 "C310" V 7150 6050 50  0000 L CNN
 F 1 "27pf" V 7350 6150 50  0000 L CNN
 F 2 "Capacitors_SMD:C_0805_HandSoldering" H 7250 6250 50  0001 C CNN
@@
 	7450 6250 7350 6250
 $Comp
-L MotorControllerParts:R_Small R302
+L MotorControllerParts:R R302
 U 1 1 5BF74546
-P 7750 6250
-F 0 "R302" V 7650 6250 50  0000 C CNN
-F 1 "390R" V 7850 6250 50  0000 C CNN
-F 2 "Resistors_SMD:R_0805_HandSoldering" H 7750 6250 50  0001 C CNN
-F 3 "~" H 7750 6250 50  0001 C CNN
-	1    7750 6250
+P 7800 6250
+F 0 "R302" V 7700 6250 50  0000 C CNN
+F 1 "330R" V 7900 6250 50  0000 C CNN
+F 2 "Resistors_SMD:R_0805_HandSoldering" H 7800 6250 50  0001 C CNN
+F 3 "http://www.yageo.com/documents/recent/PYu-RC_Group_51_RoHS_L_9.pdf" H 7800 6250 50  0001 C CNN
+F 4 "311-330CRCT-ND" H 0   0   50  0001 C CNN "Digi-key#"
+	1    7800 6250
 	0    1    1    0
 $EndComp
 Wire Wire Line
-	7850 6250 8100 6250
-Text Label 8100 5750 2    50   ~ 0
+	7950 6250 8200 6250
+Text Label 8200 5750 2    50   ~ 0
 OSC+
-Text Label 8100 6250 2    50   ~ 0
+Text Label 8200 6250 2    50   ~ 0
 OSC-
 Wire Wire Line
@@
 Connection ~ 7450 6250
 Wire Wire Line
-	8100 5750 7450 5750
+	8200 5750 7450 5750
 Connection ~ 7450 5750
 Text Label 4300 2600 0    50   ~ 0
@@
 F 1 "10K" H 2070 5605 50  0000 L CNN
 F 2 "Resistors_SMD:R_0805_HandSoldering" V 1930 5650 50  0001 C CNN
-F 3 "~" H 2000 5650 50  0001 C CNN
+F 3 "https://www.te.com/commerce/DocumentDelivery/DDEController?Action=srchrtrv&DocNm=1773204-3&DocType=DS&DocLang=English" H 2000 5650 50  0001 C CNN
+F 4 "A129761CT-ND" H 0   0   50  0001 C CNN "Digi-key#"
 	1    2000 5650
 	1    0    0    -1
@@
 F 1 "CAN_Status" H 9942 5336 50  0000 C CNN
 F 2 "LED_SMD:LED_0603_1608Metric_Pad1.05x0.95mm_HandSolder" H 9950 5500 50  0001 C CNN
-F 3 "~" H 9950 5500 50  0001 C CNN
+F 3 "https://katalog.we-online.de/pbs/datasheet/150060BS55040.pdf" H 9950 5500 50  0001 C CNN
+F 4 "732-12013-1-ND" H 0   0   50  0001 C CNN "Digi-key#"
 	1    9950 5500
 	-1   0    0    1
@@
 F 1 "SWD" H 3530 5301 50  0000 L CNN
 F 2 "Connector_PinHeader_2.54mm:PinHeader_1x06_P2.54mm_Vertical" H 3450 5400 50  0001 C CNN
-F 3 "~" H 3450 5400 50  0001 C CNN
+F 3 "https://media.digikey.com/PDF/Data%20Sheets/Sullins%20PDFs/xRxCzzzSxxN-RC_ST_11635-B.pdf" H 3450 5400 50  0001 C CNN
+F 4 "S1212EC-06-ND" H 0   0   50  0001 C CNN "Digi-key#"
 	1    3450 5400
 	1    0    0    -1
@@
 F 1 "Heartbeat" H 9942 5736 50  0000 C CNN
 F 2 "LED_SMD:LED_0603_1608Metric_Pad1.05x0.95mm_HandSolder" H 9950 5900 50  0001 C CNN
-F 3 "~" H 9950 5900 50  0001 C CNN
+F 3 "https://katalog.we-online.de/pbs/datasheet/150060RS55040.pdf" H 9950 5900 50  0001 C CNN
+F 4 "732-12015-1-ND" H 0   0   50  0001 C CNN "Digi-key#"
 	1    9950 5900
 	-1   0    0    1
@@
 F 1 "User_LED" H 9942 6136 50  0000 C CNN
 F 2 "LED_SMD:LED_0603_1608Metric_Pad1.05x0.95mm_HandSolder" H 9950 6300 50  0001 C CNN
-F 3 "~" H 9950 6300 50  0001 C CNN
+F 3 "https://katalog.we-online.com/led/datasheet/150060VS55040.pdf" H 9950 6300 50  0001 C CNN
+F 4 "732-12017-1-ND" H 0   0   50  0001 C CNN "Digi-key#"
 	1    9950 6300
 	-1   0    0    1
@@
 P 9550 6300
 F 0 "R307" V 9650 6300 50  0000 C CNN
-F 1 "510R" V 9434 6300 50  0000 C CNN
+F 1 "330R" V 9434 6300 50  0000 C CNN
 F 2 "Resistors_SMD:R_0805_HandSoldering" V 9480 6300 50  0001 C CNN
-F 3 "~" H 9550 6300 50  0001 C CNN
+F 3 "http://www.yageo.com/documents/recent/PYu-RC_Group_51_RoHS_L_9.pdf" H 9550 6300 50  0001 C CNN
+F 4 "311-330CRCT-ND" H 0   0   50  0001 C CNN "Digi-key#"
 	1    9550 6300
 	0    1    1    0
@@
 P 9550 5900
 F 0 "R306" V 9650 5900 50  0000 C CNN
-F 1 "510R" V 9434 5900 50  0000 C CNN
+F 1 "330R" V 9434 5900 50  0000 C CNN
 F 2 "Resistors_SMD:R_0805_HandSoldering" V 9480 5900 50  0001 C CNN
-F 3 "~" H 9550 5900 50  0001 C CNN
+F 3 "http://www.yageo.com/documents/recent/PYu-RC_Group_51_RoHS_L_9.pdf" H 9550 5900 50  0001 C CNN
+F 4 "311-330CRCT-ND" H 0   0   50  0001 C CNN "Digi-key#"
 	1    9550 5900
 	0    1    1    0
@@
 P 9550 5500
 F 0 "R305" V 9650 5500 50  0000 C CNN
-F 1 "510R" V 9434 5500 50  0000 C CNN
+F 1 "100R" V 9434 5500 50  0000 C CNN
 F 2 "Resistors_SMD:R_0805_HandSoldering" V 9480 5500 50  0001 C CNN
-F 3 "~" H 9550 5500 50  0001 C CNN
+F 3 "http://www.yageo.com/documents/recent/PYu-RC_Group_51_RoHS_L_9.pdf" H 9550 5500 50  0001 C CNN
+F 4 "311-100CRCT-ND" H 0   0   50  0001 C CNN "Digi-key#"
 	1    9550 5500
 	0    1    1    0
@@
 F 1 "4K7" H 9720 4005 50  0000 L CNN
 F 2 "Resistors_SMD:R_0805_HandSoldering" V 9580 4050 50  0001 C CNN
-F 3 "~" H 9650 4050 50  0001 C CNN
+F 3 "http://www.yageo.com/documents/recent/PYu-RC_Group_51_RoHS_L_9.pdf" H 9650 4050 50  0001 C CNN
+F 4 "311-4.70KCRCT-ND" H 0   0   50  0001 C CNN "Digi-key#"
 	1    9650 4050
 	1    0    0    -1
@@
 F 1 "100R" H 9720 4755 50  0000 L CNN
 F 2 "Resistors_SMD:R_0805_HandSoldering" V 9580 4800 50  0001 C CNN
-F 3 "~" H 9650 4800 50  0001 C CNN
+F 3 "http://www.yageo.com/documents/recent/PYu-RC_Group_51_RoHS_L_9.pdf" H 9650 4800 50  0001 C CNN
+F 4 "311-100CRCT-ND" H 0   0   50  0001 C CNN "Digi-key#"
 	1    9650 4800
 	1    0    0    -1
@@
 F 1 "User USART" H 9750 2900 50  0000 L CNN
 F 2 "Connector_PinHeader_2.54mm:PinHeader_1x03_P2.54mm_Vertical" H 9950 3100 50  0001 C CNN
-F 3 "~" H 9950 3100 50  0001 C CNN
+F 3 "https://media.digikey.com/PDF/Data%20Sheets/Sullins%20PDFs/xRxCzzzSxxN-RC_ST_11635-B.pdf" H 9950 3100 50  0001 C CNN
+F 4 "S1212EC-03-ND" H 0   0   50  0001 C CNN "Digi-key#"
 	1    9950 3100
 	1    0    0    -1

Commit message: PCB rev 1.1 -Fixed the TMC4671 footprint (use the Digi-Key layout) -Fixed the USB pull up issue for using the DFU bootloader -Fixed the orientation of the Hall sensor connector -Added a PTC on the hall effect sensor line -Added a 5v jumper for the CAN port
Parts:
- added R308: 1K5, Resistor_SMD:R_0805_2012Metric, symbol MotorControllerParts:R_Small
Connections:
- net labels added: +3V3
- wire segments 183 -> 186
Other:
- note added: "1.5 KOhm pull up: \nenable USB programming"
Changed lines of the file:
@@
 Wire Wire Line
 	6800 4200 6100 4200
-Text Label 6800 2500 2    50   ~ 0
+Text Label 7550 2500 2    50   ~ 0
 USB_D+
-Text Label 6800 2400 2    50   ~ 0
+Text Label 7550 2400 2    50   ~ 0
 USB_D-
 Wire Wire Line
-	6800 2500 6100 2500
-Wire Wire Line
-	6800 2400 6100 2400
+	7550 2400 6100 2400
 Text Label 6800 1700 2    50   ~ 0
 A_Out1
@@
 NoConn ~ 4700 4400
 NoConn ~ 6100 2300
+$Comp
+L MotorControllerParts:+3V3 #PWR0319
+U 1 1 5C70AB9B
+P 7000 2000
+F 0 "#PWR0319" H 7000 1850 50  0001 C CNN
+F 1 "+3V3" H 7015 2173 50  0000 C CNN
+F 2 "" H 7000 2000 50  0001 C CNN
+F 3 "" H 7000 2000 50  0001 C CNN
+	1    7000 2000
+	1    0    0    -1
+$EndComp
+$Comp
+L MotorControllerParts:R_Small R308
+U 1 1 5C70AD3D
+P 7000 2150
+F 0 "R308" H 7059 2196 50  0000 L CNN
+F 1 "1K5" H 7059 2105 50  0000 L CNN
+F 2 "Resistor_SMD:R_0805_2012Metric" H 7000 2150 50  0001 C CNN
+F 3 "" H 7000 2150 50  0001 C CNN
+	1    7000 2150
+	1    0    0    -1
+$EndComp
+Wire Wire Line
+	7000 2050 7000 2000
+Wire Wire Line
+	6100 2500 7000 2500
+Wire Wire Line
+	7000 2250 7000 2500
+Connection ~ 7000 2500
+Wire Wire Line
+	7000 2500 7550 2500
+Text Notes 7300 2200 0    50   ~ 0
+1.5 KOhm pull up: \nenable USB programming
 $EndSCHEMATC
